File: LightRail_LPO_1.6T.kicad_pcb (KiCad board)
At the start: 10 copper layers, 218 parts, among them J1 MPO-24, U1 TFLN_Mod_Gen3_8CH, U2 NeoPhotonics_1550nm_DFB, U3 Si5395A, U4 AD5684R, U5 MAX3669, U6 TPS7A2018, U7 TPS54360, U8 MPT5000

Commit message: feat: implement dual AI Compute Node with TFLN photonic integration
- Add hierarchical sub-sheets: AI_Core (SoC BGA 2500-pin, TFLN interface),
  Memory (DDR5 DIMM 288-pin fly-by topology), VRM (24-phase DrMOS array)
- Update root schematic with dual compute unit hierarchy (2x AI_Core,
  2x VRM, 32x Memory sheets)
- Add net classes: TFLN_RF (0.15mm/0.20mm diff), PCIe_Gen6 (0.12mm/0.18mm),
  DDR5_Data (0.10mm/0.15mm micro-via), PWR_CORE (2.0mm+)
- Create custom footprints: BGA-2500 (50x50, 0.8mm pitch), TFLN_PIC
  (periphery pads, optical keepout center), DrMOS PowerPAK 8x8mm,
  DDR5 DIMM 288-pin connector
- Update PCB: TFLN keepout zones, VRM V_core copper pours on internal
  layers, GND reference plane, DDR5 fly-by routing structures
- Place AI SoC BGA, TFLN PIC, and DrMOS footprints for both units
- Update project rev to 4.0, date to 2026-04-11

Co-Authored-By: Bola Olatunji <bola.olatunji@ai.lightos.sh>
Parts:
- added U101: AI_SoC_U0, LightRail:BGA-2500_40x40mm_P0.8mm, F.Cu at (42.0, 50.0)
- added U102: TFLN_PIC_U0, LightRail:TFLN_PIC_Periphery, F.Cu at (55.0, 20.0)
- added U201: AI_SoC_U1, LightRail:BGA-2500_40x40mm_P0.8mm, F.Cu at (126.0, 50.0)
- added U202: TFLN_PIC_U1, LightRail:TFLN_PIC_Periphery, F.Cu at (113.0, 20.0)
- added U302: ISL99390, LightRail:DrMOS_PowerPAK_8x8mm, F.Cu at (10.0, 85.0)
- added U303: ISL99390, LightRail:DrMOS_PowerPAK_8x8mm, F.Cu at (22.0, 85.0)
- added U304: ISL99390, LightRail:DrMOS_PowerPAK_8x8mm, F.Cu at (34.0, 85.0)
- added U305: ISL99390, LightRail:DrMOS_PowerPAK_8x8mm, F.Cu at (46.0, 85.0)
- added U306: ISL99390, LightRail:DrMOS_PowerPAK_8x8mm, F.Cu at (58.0, 85.0)
- added U307: ISL99390, LightRail:DrMOS_PowerPAK_8x8mm, F.Cu at (70.0, 85.0)
- added U326: ISL99390, LightRail:DrMOS_PowerPAK_8x8mm, F.Cu at (94.0, 85.0)
- added U327: ISL99390, LightRail:DrMOS_PowerPAK_8x8mm, F.Cu at (106.0, 85.0)
- added U328: ISL99390, LightRail:DrMOS_PowerPAK_8x8mm, F.Cu at (118.0, 85.0)
- added U329: ISL99390, LightRail:DrMOS_PowerPAK_8x8mm, F.Cu at (130.0, 85.0)
- added U330: ISL99390, LightRail:DrMOS_PowerPAK_8x8mm, F.Cu at (142.0, 85.0)
- added U331: ISL99390, LightRail:DrMOS_PowerPAK_8x8mm, F.Cu at (154.0, 85.0)
Routing:
- net (no net): track 0.00 -> 216.0 mm
- added copper zone on In7.Cu, net GND
- added copper zone on In3.Cu, net V_CORE_U0
- added copper zone on In4.Cu, net V_CORE_U0
- added copper zone on In5.Cu, net V_CORE_U1
- added copper zone on In6.Cu, net V_CORE_U1
Other:
- board text added: "AI COMPUTE UNIT 0"
- board text added: "AI COMPUTE UNIT 1"
- board text added: "DDR5 DIMM SLOTS"
- board text added: "LightRail LPO 1.6T Dual AI Compute Node Rev 4.0"
- board text added: "TFLN OPTICAL ENGINE"
- board text added: "VRM 24-PHASE"

Commit message: fix: correct net IDs on power zones, DDR5 traces, and via_diameter DRC violation
- V_CORE_U0 zones (In3.Cu, In4.Cu): net 0 → net 164
- V_CORE_U1 zones (In5.Cu, In6.Cu): net 0 → net 165
- GND zone (In7.Cu): net 0 → net 1 (matching existing GND zones)
- DDR5 fly-by CK segments: net 0 → net 152/153 (U0) and 160/161 (U1)
- DDR5_Data net class via_diameter: 0.25mm → 0.3mm (meets min_via_diameter)

Co-Authored-By: Bola Olatunji <bola.olatunji@ai.lightos.sh>
Routing:
- net (no net): track 216.0 -> 0.00 mm
- net DDR5_U1_CK_P: track 0.00 -> 56.0 mm
- net DDR5_U0_CK_P: track 0.00 -> 56.0 mm
- net DDR5_U1_CK_N: track 0.00 -> 52.0 mm
- net DDR5_U0_CK_N: track 0.00 -> 52.0 mm
Changed lines of the file:
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@@
     )
   )
-  (zone (net 0) (net_name "V_CORE_U0") (layer "In3.Cu") (hatch edge 0.508)
+  (zone (net 164) (net_name "V_CORE_U0") (layer "In3.Cu") (hatch edge 0.508)
     (connect_pads thru_hole_only (clearance 0.3))
     (fill yes (thermal_gap 0) (thermal_bridge_width 1.0))
@@
     )
   )
-  (zone (net 0) (net_name "V_CORE_U0") (layer "In4.Cu") (hatch edge 0.508)
+  (zone (net 164) (net_name "V_CORE_U0") (layer "In4.Cu") (hatch edge 0.508)
     (connect_pads thru_hole_only (clearance 0.3))
     (fill yes (thermal_gap 0) (thermal_bridge_width 1.0))
@@
     )
   )
-  (zone (net 0) (net_name "V_CORE_U1") (layer "In5.Cu") (hatch edge 0.508)
+  (zone (net 165) (net_name "V_CORE_U1") (layer "In5.Cu") (hatch edge 0.508)
     (connect_pads thru_hole_only (clearance 0.3))
     (fill yes (thermal_gap 0) (thermal_bridge_width 1.0))
@@
     )
   )
-  (zone (net 0) (net_name "V_CORE_U1") (layer "In6.Cu") (hatch edge 0.508)
+  (zone (net 165) (net_name "V_CORE_U1") (layer "In6.Cu") (hatch edge 0.508)
     (connect_pads thru_hole_only (clearance 0.3))
     (fill yes (thermal_gap 0) (thermal_bridge_width 1.0))
@@
     )
   )
-  (zone (net 0) (net_name "GND") (layer "In7.Cu") (hatch edge 0.508)
+  (zone (net 1) (net_name "GND") (layer "In7.Cu") (hatch edge 0.508)
     (connect_pads thru_hole_only (clearance 0.3))
     (fill yes (thermal_gap 0.508) (thermal_bridge_width 0.508))
@@
   )
   ;; === DDR5 FLY-BY TOPOLOGY ROUTING STRUCTURES ===
-  (segment (start 15.0 72) (end 29.0 72) (width 0.1) (layer "In1.Cu") (net 0))
-  (segment (start 15.0 74) (end 28.0 74) (width 0.1) (layer "In1.Cu") (net 0))
-  (segment (start 30.0 72) (end 44.0 72) (width 0.1) (layer "In1.Cu") (net 0))
-  (segment (start 30.0 74) (end 43.0 74) (width 0.1) (layer "In1.Cu") (net 0))
-  (segment (start 45.0 72) (end 59.0 72) (width 0.1) (layer "In1.Cu") (net 0))
-  (segment (start 45.0 74) (end 58.0 74) (width 0.1) (layer "In1.Cu") (net 0))
-  (segment (start 60.0 72) (end 74.0 72) (width 0.1) (layer "In1.Cu") (net 0))
-  (segment (start 60.0 74) (end 73.0 74) (width 0.1) (layer "In1.Cu") (net 0))
-  (segment (start 90.0 72) (end 104.0 72) (width 0.1) (layer "In1.Cu") (net 0))
-  (segment (start 90.0 74) (end 103.0 74) (width 0.1) (layer "In1.Cu") (net 0))
-  (segment (start 105.0 72) (end 119.0 72) (width 0.1) (layer "In1.Cu") (net 0))
-  (segment (start 105.0 74) (end 118.0 74) (width 0.1) (layer "In1.Cu") (net 0))
-  (segment (start 120.0 72) (end 134.0 72) (width 0.1) (layer "In1.Cu") (net 0))
-  (segment (start 120.0 74) (end 133.0 74) (width 0.1) (layer "In1.Cu") (net 0))
-  (segment (start 135.0 72) (end 149.0 72) (width 0.1) (layer "In1.Cu") (net 0))
-  (segment (start 135.0 74) (end 148.0 74) (width 0.1) (layer "In1.Cu") (net 0))
+  (segment (start 15.0 72) (end 29.0 72) (width 0.1) (layer "In1.Cu") (net 152))
+  (segment (start 15.0 74) (end 28.0 74) (width 0.1) (layer "In1.Cu") (net 153))
+  (segment (start 30.0 72) (end 44.0 72) (width 0.1) (layer "In1.Cu") (net 152))
+  (segment (start 30.0 74) (end 43.0 74) (width 0.1) (layer "In1.Cu") (net 153))
+  (segment (start 45.0 72) (end 59.0 72) (width 0.1) (layer "In1.Cu") (net 152))
+  (segment (start 45.0 74) (end 58.0 74) (width 0.1) (layer "In1.Cu") (net 153))
+  (segment (start 60.0 72) (end 74.0 72) (width 0.1) (layer "In1.Cu") (net 152))
+  (segment (start 60.0 74) (end 73.0 74) (width 0.1) (layer "In1.Cu") (net 153))
+  (segment (start 90.0 72) (end 104.0 72) (width 0.1) (layer "In1.Cu") (net 160))
+  (segment (start 90.0 74) (end 103.0 74) (width 0.1) (layer "In1.Cu") (net 161))
+  (segment (start 105.0 72) (end 119.0 72) (width 0.1) (layer "In1.Cu") (net 160))
+  (segment (start 105.0 74) (end 118.0 74) (width 0.1) (layer "In1.Cu") (net 161))
+  (segment (start 120.0 72) (end 134.0 72) (width 0.1) (layer "In1.Cu") (net 160))
+  (segment (start 120.0 74) (end 133.0 74) (width 0.1) (layer "In1.Cu") (net 161))
+  (segment (start 135.0 72) (end 149.0 72) (width 0.1) (layer "In1.Cu") (net 160))
+  (segment (start 135.0 74) (end 148.0 74) (width 0.1) (layer "In1.Cu") (net 161))
   ;; === AI SoC BGA AND TFLN PIC FOOTPRINTS ===
   (footprint "LightRail:BGA-2500_40x40mm_P0.8mm" (layer "F.Cu")

Commit message: fix(pcb,docs): address Devin Review findings
- Stackup: V_CORE_U1 planes (In5.Cu, In6.Cu) go from 0.5 oz to 2 oz so
  U1 matches U0 PDN impedance (previous 4:1 asymmetry would have
  violated the 10 mV IR-drop target for V_CORE_U1)
- .kicad_pcb stackup: bump In5.Cu / In6.Cu thickness 0.0175 -> 0.035 mm
- gerber_layers.txt In5/In6 re-labelled as V_CORE_U1 planes (the zones
  there already carry net 165 = V_CORE_U1; docs now match PCB)
- Note added to Stackup.md that DDR5 byte lanes 2-3 cannot live on
  In5/In6 in the 10-layer scaffold -> tape-out 22-24 layer target
- DDR5 CK fly-by segments moved from In1.Cu (GND reference plane) to
  In2.Cu (designated DDR5 stripline layer); P/N endpoints now equal
  length to remove the 1 mm intra-pair skew
- TFLN optical keep-outs repositioned: previous polygons (40,35)-(70,55)
  and (98,35)-(128,55) overlapped the BGA-2500 pad fields at (55,45)
  and (110,45). New keep-outs are at the front-panel fiber-exit region
  and mirrored on B.Cu
- DDR5_Data net class: via_diameter 0.3 -> 0.35 mm (safe margin above
  the project-wide min_via_diameter of 0.3 mm), microvia_diameter
  0.25 -> 0.3 mm
- DRC rule ddr5_ca_stripline_only: use KiCad 8 regex (=~) against the
  real net names (DDR5_U0_CK_P etc.) instead of short literals that
  never matched
- Added rule ddr5_ck_ca_length_match (skew <= 0.05 mm) as a warning
- README.md: add Rev 4.1 entry + 'Residual items flagged by Devin
  Review that still require human work' section covering the
  schematic-side fixes (VDD_IO / TFLN_CLK / DDR5 / VID sheet pins)
  that should not be edited via text surgery

Co-Authored-By: Bola Olatunji <bola.olatunji@ai.lightos.sh>
Routing:
- net DDR5_U1_CK_N: track 52.0 -> 56.0 mm
- net DDR5_U0_CK_N: track 52.0 -> 56.0 mm
Changed lines of the file:
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@@
       (layer "In4.Cu" (type "copper") (thickness 0.035))
       (layer "dielectric 5" (type "prepreg") (thickness 0.0994) (material "Megtron-7") (epsilon_r 3.3) (loss_tangent 0.002))
-      (layer "In5.Cu" (type "copper") (thickness 0.0175))
+      (layer "In5.Cu" (type "copper") (thickness 0.035))
       (layer "dielectric 6" (type "core") (thickness 0.2) (material "Megtron-7") (epsilon_r 3.3) (loss_tangent 0.002))
-      (layer "In6.Cu" (type "copper") (thickness 0.0175))
+      (layer "In6.Cu" (type "copper") (thickness 0.035))
       (layer "dielectric 7" (type "prepreg") (thickness 0.0994) (material "Megtron-7") (epsilon_r 3.3) (loss_tangent 0.002))
       (layer "In7.Cu" (type "copper") (thickness 0.035))
@@
   (net 168 "PGOOD_U1")
   ;; === TFLN KEEPOUT ZONES (no copper under optical fiber paths) ===
+  ;; TFLN optical fiber-exit keep-outs (front-panel region, not over BGA).
+  ;; Dimensions are a scaffold: human layout engineer must reposition
+  ;; these to match final SoC placement before tape-out.
   (zone (net 0) (net_name "") (layer "F.Cu") (hatch edge 0.508)
     (connect_pads (clearance 0))
@@
     (polygon
       (pts
-        (xy 40 35)
-        (xy 70 35)
-        (xy 70 55)
-        (xy 40 55)
+        (xy 10 5)
+        (xy 40 5)
+        (xy 40 20)
+        (xy 10 20)
       )
     )
@@
     (polygon
       (pts
-        (xy 98 35)
-        (xy 128 35)
-        (xy 128 55)
-        (xy 98 55)
+        (xy 128 5)
+        (xy 158 5)
+        (xy 158 20)
+        (xy 128 20)
+      )
+    )
+  )
+  ;; Mirrored keepouts on B.Cu so bottom-side routing also respects the
+  ;; front-panel optical-fiber exit.
+  (zone (net 0) (net_name "") (layer "B.Cu") (hatch edge 0.508)
+    (connect_pads (clearance 0))
+    (fill (thermal_gap 0.508) (thermal_bridge_width 0.508))
+    (keepout (tracks not_allowed) (vias not_allowed) (pads not_allowed) (copperpour not_allowed) (footprints allowed))
+    (polygon
+      (pts
+        (xy 10 5)
+        (xy 40 5)
+        (xy 40 20)
+        (xy 10 20)
+      )
+    )
+  )
+  (zone (net 0) (net_name "") (layer "B.Cu") (hatch edge 0.508)
+    (connect_pads (clearance 0))
+    (fill (thermal_gap 0.508) (thermal_bridge_width 0.508))
+    (keepout (tracks not_allowed) (vias not_allowed) (pads not_allowed) (copperpour not_allowed) (footprints allowed))
+    (polygon
+      (pts
+        (xy 128 5)
+        (xy 158 5)
+        (xy 158 20)
+        (xy 128 20)
       )
     )
@@
   )
   ;; === DDR5 FLY-BY TOPOLOGY ROUTING STRUCTURES ===
-  (segment (start 15.0 72) (end 29.0 72) (width 0.1) (layer "In1.Cu") (net 152))
-  (segment (start 15.0 74) (end 28.0 74) (width 0.1) (layer "In1.Cu") (net 153))
-  (segment (start 30.0 72) (end 44.0 72) (width 0.1) (layer "In1.Cu") (net 152))
-  (segment (start 30.0 74) (end 43.0 74) (width 0.1) (layer "In1.Cu") (net 153))
-  (segment (start 45.0 72) (end 59.0 72) (width 0.1) (layer "In1.Cu") (net 152))
-  (segment (start 45.0 74) (end 58.0 74) (width 0.1) (layer "In1.Cu") (net 153))
-  (segment (start 60.0 72) (end 74.0 72) (width 0.1) (layer "In1.Cu") (net 152))
-  (segment (start 60.0 74) (end 73.0 74) (width 0.1) (layer "In1.Cu") (net 153))
-  (segment (start 90.0 72) (end 104.0 72) (width 0.1) (layer "In1.Cu") (net 160))
-  (segment (start 90.0 74) (end 103.0 74) (width 0.1) (layer "In1.Cu") (net 161))
-  (segment (start 105.0 72) (end 119.0 72) (width 0.1) (layer "In1.Cu") (net 160))
-  (segment (start 105.0 74) (end 118.0 74) (width 0.1) (layer "In1.Cu") (net 161))
-  (segment (start 120.0 72) (end 134.0 72) (width 0.1) (layer "In1.Cu") (net 160))
-  (segment (start 120.0 74) (end 133.0 74) (width 0.1) (layer "In1.Cu") (net 161))
-  (segment (start 135.0 72) (end 149.0 72) (width 0.1) (layer "In1.Cu") (net 160))
-  (segment (start 135.0 74) (end 148.0 74) (width 0.1) (layer "In1.Cu") (net 161))
+  ;; Stripline on In2.Cu between GND (In1.Cu) above and V_CORE_U0 (In3.Cu) below.
+  ;; P/N endpoints are equal to keep intra-pair skew ≈ 0 mm.
+  (segment (start 15.0 72) (end 29.0 72) (width 0.1) (layer "In2.Cu") (net 152))
+  (segment (start 15.0 74) (end 29.0 74) (width 0.1) (layer "In2.Cu") (net 153))
+  (segment (start 30.0 72) (end 44.0 72) (width 0.1) (layer "In2.Cu") (net 152))
+  (segment (start 30.0 74) (end 44.0 74) (width 0.1) (layer "In2.Cu") (net 153))
+  (segment (start 45.0 72) (end 59.0 72) (width 0.1) (layer "In2.Cu") (net 152))
+  (segment (start 45.0 74) (end 59.0 74) (width 0.1) (layer "In2.Cu") (net 153))
+  (segment (start 60.0 72) (end 74.0 72) (width 0.1) (layer "In2.Cu") (net 152))
+  (segment (start 60.0 74) (end 74.0 74) (width 0.1) (layer "In2.Cu") (net 153))
+  (segment (start 90.0 72) (end 104.0 72) (width 0.1) (layer "In2.Cu") (net 160))
+  (segment (start 90.0 74) (end 104.0 74) (width 0.1) (layer "In2.Cu") (net 161))
+  (segment (start 105.0 72) (end 119.0 72) (width 0.1) (layer "In2.Cu") (net 160))
+  (segment (start 105.0 74) (end 119.0 74) (width 0.1) (layer "In2.Cu") (net 161))
+  (segment (start 120.0 72) (end 134.0 72) (width 0.1) (layer "In2.Cu") (net 160))
+  (segment (start 120.0 74) (end 134.0 74) (width 0.1) (layer "In2.Cu") (net 161))
+  (segment (start 135.0 72) (end 149.0 72) (width 0.1) (layer "In2.Cu") (net 160))
+  (segment (start 135.0 74) (end 149.0 74) (width 0.1) (layer "In2.Cu") (net 161))
   ;; === AI SoC BGA AND TFLN PIC FOOTPRINTS ===
   (footprint "LightRail:BGA-2500_40x40mm_P0.8mm" (layer "F.Cu")
