File: LightRail_LPO_1.6T.kicad_pcb (KiCad board)
At the start: 10 copper layers, 168 x 105 mm, 234 parts, among them J1 MPO-24, U1 TFLN_Mod_Gen3_8CH, U101 AI_SoC_U0, U102 TFLN_PIC_U0, U2 NeoPhotonics_1550nm_DFB, U201 AI_SoC_U1, U202 TFLN_PIC_U1, U3 Si5395A, U302 ISL99390, U303 ISL99390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

Commit message: fix(pcb,docs): remove conflicting plane zones; fix impedance refs; thickness 1.86->1.81
Three Devin Review findings on the stackup-symmetry follow-up:

1. Conflicting zones on V_CORE layers. The previous scaffold put
   board-wide +12V on In3.Cu, +3V3 on In4.Cu, and GND on In5.Cu.
   After the recent re-tasking of In3..In6 as dedicated V_CORE_U0 /
   V_CORE_U1 planes (with explicit V_CORE_U0 zones on In3+In4 and
   V_CORE_U1 zones on In5+In6), those old full-board zones would
   fight the new zones on the same layers at refill time and either
   produce DRC net-short violations or carve clearance holes that
   break V_CORE plane continuity under 1000 A load. Removed all three
   stale zones. In1.Cu (GND), In7.Cu (GND), and B.Cu (GND) retained.

2. General header thickness 1.86 -> 1.81 mm. The stackup-symmetry
   commit computed 1.81 mm and propagated it to docs/Stackup.md and
   docs/Fab_Notes.md but missed the (general (thickness)) field in
   the PCB header (my bad — an Edit that looked applied in the tool
   output didn't make it into the staged diff). Fix now so KiCad's
   3D viewer, ODB++ header, and parser-driven checks all see 1.81.

3. Impedance table incorrectly called In3.Cu a GND reference. In3 is
   the V_CORE_U0 plane, not GND, so striplines routed between In1
   (GND) and In3 (V_CORE) actually see an asymmetric reference pair.
   Updated the Reference-plane column for SERDES_100G_PAM4, PCIe_Gen6,
   RF_50OHM_DIFF, DDR5_Data, and single-ended DDR5 to read
   'GND (In1) / V_CORE (In3)' and added an explicit 'Asymmetric
   stripline note' below the table explaining that V_CORE is valid as
   an AC reference (GND-decoupled at the BGA via the bulk + MLCC
   network) but the fab must solve the asymmetric stack, not assume
   symmetric GND-GND. TFLN_RF (microstrip) and USB3/USB4 (microstrip)
   untouched — their references on F.Cu / In1 are unchanged.

Co-Authored-By: Bola Olatunji <bola.olatunji@ai.lightos.sh>
Routing:
- removed copper zone on In3.Cu, net +12V
- removed copper zone on In4.Cu, net +3V3
- removed copper zone on In5.Cu, net GND
Changed lines of the file:
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@@
 (kicad_pcb (version 20211014) (generator pcbnew)
   (general
-    (thickness 1.86)
+    (thickness 1.81)
   )
   (paper "A4")
@@
     ))
   )
-  (zone (net 1) (net_name "GND") (layer "In5.Cu") (hatch edge 0.508)
-    (connect_pads (clearance 0.15))
-    (min_thickness 0.1)
-    (fill yes (thermal_gap 0.3) (thermal_bridge_width 0.3))
-    (polygon (pts
-      (xy 0 0) (xy 168.0 0) (xy 168.0 100.0) (xy 0 100.0)
-    ))
-  )
   (zone (net 1) (net_name "GND") (layer "B.Cu") (hatch edge 0.508)
     (connect_pads (clearance 0.15))
@@
     (fill yes (thermal_gap 0.3) (thermal_bridge_width 0.3))
     (polygon (pts
-      (xy 0 0) (xy 168.0 0) (xy 168.0 100.0) (xy 0 100.0)
-    ))
-  )
-  (zone (net 2) (net_name "+12V") (layer "In3.Cu") (hatch edge 0.508)
-    (connect_pads (clearance 0.2))
-    (min_thickness 0.15)
-    (fill yes (thermal_gap 0.3) (thermal_bridge_width 0.3))
-    (polygon (pts
-      (xy 0 0) (xy 168.0 0) (xy 168.0 100.0) (xy 0 100.0)
-    ))
-  )
-  (zone (net 3) (net_name "+3V3") (layer "In4.Cu") (hatch edge 0.508)
-    (connect_pads (clearance 0.2))
-    (min_thickness 0.15)
-    (fill yes (thermal_gap 0.3) (thermal_bridge_width 0.3))
-    (polygon (pts

Commit message: fix(pcb): V_CORE plane coverage, TFLN keepout placement, DDR5 CK contiguity
Three Devin Review findings on the PCB scaffold zones and routes:

1. V_CORE plane zones covered only the bottom 25 % of each BGA-2500
   footprint. U101 lives at (42,50) with \u00b120 mm body (x=22..62,
   y=30..70), but the V_CORE_U0 zone on In3.Cu/In4.Cu was
   (5,60)-(78,95) — it only overlapped y=60..70 of the SoC, i.e. a
   10 mm-wide strip at the BGA south edge. All V_CORE balls in the
   upper 75 % of the BGA had no plane beneath them on a power layer,
   forcing all 1000 A through a thin strip and making the <=10 mV /
   <=0.5 m\u03a9 PDN target in SI_PI_Thermal_Plan.md impossible to meet.
   Extended V_CORE_U0 y-range to (5,25)-(78,95) so the whole U101 BGA
   sits over the plane. Same fix for V_CORE_U1 on In5.Cu/In6.Cu:
   (90,60)-(163,95) -> (90,25)-(163,95), covering U201 at (126,50).

2. TFLN optical keepout zones were in the wrong place. U102 is at
   (55,20) and U202 at (113,20), but the four keepout polygons were
   drawn at (10..40, 5..20) and (128..158, 5..20) — zero x-axis
   overlap with either PIC. The F.Cu / In1.Cu GND flood would have
   poured copper straight through the optical waveguide region under
   both TFLN die. Moved all four keepouts to (47..63, 12..28) and
   (105..121, 12..28) so they sit directly over the PICs
   (\u00b18 mm body + 0 mm keepout margin as a scaffold intent; the
   tape-out keepout should be the PIC's published optical keep-clear
   polygon, typically \u00b18.5 mm).

3. DDR5 CK segments had 1 mm open gaps between consecutive stubs.
   Net 152 had end=29 then start=30; end=44 then start=45; end=59
   then start=60. Same pattern on nets 153, 160, 161. Each fly-by
   stub was therefore 4x 14 mm disconnected segments instead of one
   continuous 59 mm trace. Closed the gaps by extending each
   segment's end to the next segment's start — 29->30, 44->45,
   59->60 on the U0 nets; 104->105, 119->120, 134->135 on the U1
   nets. CK_P and CK_N now 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
Routing:
- net DDR5_U1_CK_P: track 56.0 -> 59.0 mm
- net DDR5_U1_CK_N: track 56.0 -> 59.0 mm
- net DDR5_U0_CK_P: track 56.0 -> 59.0 mm
- net DDR5_U0_CK_N: track 56.0 -> 59.0 mm
Changed lines of the file:
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@@
     (polygon
       (pts
-        (xy 10 5)
-        (xy 40 5)
-        (xy 40 20)
-        (xy 10 20)
+        (xy 47 12)
+        (xy 63 12)
+        (xy 63 28)
+        (xy 47 28)
       )
     )
@@
     (polygon
       (pts
-        (xy 128 5)
-        (xy 158 5)
-        (xy 158 20)
-        (xy 128 20)
+        (xy 105 12)
+        (xy 121 12)
+        (xy 121 28)
+        (xy 105 28)
       )
     )
@@
     (polygon
       (pts
-        (xy 10 5)
-        (xy 40 5)
-        (xy 40 20)
-        (xy 10 20)
+        (xy 47 12)
+        (xy 63 12)
+        (xy 63 28)
+        (xy 47 28)
       )
     )
@@
     (polygon
       (pts
-        (xy 128 5)
-        (xy 158 5)
-        (xy 158 20)
-        (xy 128 20)
+        (xy 105 12)
+        (xy 121 12)
+        (xy 121 28)
+        (xy 105 28)
       )
     )
@@
     (polygon
       (pts
-        (xy 5 60)
-        (xy 78 60)
+        (xy 5 25)
+        (xy 78 25)
         (xy 78 95)
         (xy 5 95)
@@
     (polygon
       (pts
-        (xy 5 60)
-        (xy 78 60)
+        (xy 5 25)
+        (xy 78 25)
         (xy 78 95)
         (xy 5 95)
@@
     (polygon
       (pts
-        (xy 90 60)
-        (xy 163 60)
+        (xy 90 25)
+        (xy 163 25)
         (xy 163 95)
         (xy 90 95)
@@
     (polygon
       (pts
-        (xy 90 60)
-        (xy 163 60)
+        (xy 90 25)
+        (xy 163 25)
         (xy 163 95)
         (xy 90 95)
@@
     )
   )
-  (segment (start 15.0 72) (end 29.0 72) (width 0.1) (layer "In2.Cu") (net 152))
-  (segment (start 15.0 72.25) (end 29.0 72.25) (width 0.1) (layer "In2.Cu") (net 153))
-  (segment (start 30.0 72) (end 44.0 72) (width 0.1) (layer "In2.Cu") (net 152))
-  (segment (start 30.0 72.25) (end 44.0 72.25) (width 0.1) (layer "In2.Cu") (net 153))
-  (segment (start 45.0 72) (end 59.0 72) (width 0.1) (layer "In2.Cu") (net 152))
-  (segment (start 45.0 72.25) (end 59.0 72.25) (width 0.1) (layer "In2.Cu") (net 153))
+  (segment (start 15.0 72) (end 30.0 72) (width 0.1) (layer "In2.Cu") (net 152))
+  (segment (start 15.0 72.25) (end 30.0 72.25) (width 0.1) (layer "In2.Cu") (net 153))
+  (segment (start 30.0 72) (end 45.0 72) (width 0.1) (layer "In2.Cu") (net 152))
+  (segment (start 30.0 72.25) (end 45.0 72.25) (width 0.1) (layer "In2.Cu") (net 153))
+  (segment (start 45.0 72) (end 60.0 72) (width 0.1) (layer "In2.Cu") (net 152))
+  (segment (start 45.0 72.25) (end 60.0 72.25) (width 0.1) (layer "In2.Cu") (net 153))
   (segment (start 60.0 72) (end 74.0 72) (width 0.1) (layer "In2.Cu") (net 152))
   (segment (start 60.0 72.25) (end 74.0 72.25) (width 0.1) (layer "In2.Cu") (net 153))
-  (segment (start 90.0 72) (end 104.0 72) (width 0.1) (layer "In2.Cu") (net 160))
-  (segment (start 90.0 72.25) (end 104.0 72.25) (width 0.1) (layer "In2.Cu") (net 161))
-  (segment (start 105.0 72) (end 119.0 72) (width 0.1) (layer "In2.Cu") (net 160))
-  (segment (start 105.0 72.25) (end 119.0 72.25) (width 0.1) (layer "In2.Cu") (net 161))
-  (segment (start 120.0 72) (end 134.0 72) (width 0.1) (layer "In2.Cu") (net 160))
-  (segment (start 120.0 72.25) (end 134.0 72.25) (width 0.1) (layer "In2.Cu") (net 161))
+  (segment (start 90.0 72) (end 105.0 72) (width 0.1) (layer "In2.Cu") (net 160))
+  (segment (start 90.0 72.25) (end 105.0 72.25) (width 0.1) (layer "In2.Cu") (net 161))
+  (segment (start 105.0 72) (end 120.0 72) (width 0.1) (layer "In2.Cu") (net 160))
+  (segment (start 105.0 72.25) (end 120.0 72.25) (width 0.1) (layer "In2.Cu") (net 161))
+  (segment (start 120.0 72) (end 135.0 72) (width 0.1) (layer "In2.Cu") (net 160))
+  (segment (start 120.0 72.25) (end 135.0 72.25) (width 0.1) (layer "In2.Cu") (net 161))
   (segment (start 135.0 72) (end 149.0 72) (width 0.1) (layer "In2.Cu") (net 160))
   (segment (start 135.0 72.25) (end 149.0 72.25) (width 0.1) (layer "In2.Cu") (net 161))

Commit message: fix(pcb,sch,docs): Unit 1 In3 GND island; DDR5 diff Z 85->80 Ohm
Two Devin Review findings:

1. Unit 1 DDR5 CK (nets 160/161 on In2.Cu, x=90..149) had no lower
   reference plane. V_CORE_U0 on In3.Cu only covers x=5..78 (Unit 0
   region), and V_CORE_U1 is on In5/In6 — two dielectric layers below
   In2, too far to act as a return-path reference. Previously the
   deleted board-wide +12V zone on In3.Cu was accidentally serving
   that role; once it was removed for the V_CORE re-tasking, Unit 1
   signals on In2.Cu were left as one-sided microstrip referenced
   only to In1.Cu GND, which pushes their differential impedance to
   ~120 Ohm instead of the 80 Ohm target.

   Fix: added two GND fill zones (net 1) at In3.Cu and In4.Cu
   covering Unit 1 region (x=80..168, y=0..100). In3 GND restores
   the lower reference for DDR5 / PCIe signals on In2.Cu under
   Unit 1, giving a symmetric GND/GND stripline (vs Unit 0's
   asymmetric GND/V_CORE). In4 GND mirrors this for PDN plane
   continuity under Unit 1's BGA and keeps the stackup symmetric
   (V_CORE_U0 island on In3/In4 left half, GND island on In3/In4
   right half). Updated docs/Stackup.md §2 Asymmetric stripline
   note to document the two-region reference strategy explicitly.

2. Memory.kicad_sch said '85 Ohm differential for DQ/DQS' (lines
   13 and 159) while docs/Stackup.md:79 specifies 80 Ohm diff for
   DDR5_Data. The 5 Ohm gap matters because a 2D field solver will
   produce different trace widths/gaps for 80 vs 85 Ohm — a fab
   following one doc will fail the other's spec. Standardised on
   80 Ohm diff / 40 Ohm SE (JEDEC JESD79-5 baseline for DDR5-5600)
   in both Memory.kicad_sch comment lines.

Co-Authored-By: Bola Olatunji <bola.olatunji@ai.lightos.sh>
Routing:
- added copper zone on In3.Cu, net GND
- added copper zone on In4.Cu, net GND
Changed lines of the file:
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@@
+    )
+  )
+  (zone (net 1) (net_name "GND") (layer "In3.Cu") (hatch edge 0.508)
+    (connect_pads thru_hole_only (clearance 0.3))
+    (fill yes (thermal_gap 0.508) (thermal_bridge_width 0.508))
+    (polygon
+      (pts
+        (xy 80 0)
+        (xy 168 0)
+        (xy 168 100)
+        (xy 80 100)
+      )
+    )
+  )
+  (zone (net 1) (net_name "GND") (layer "In4.Cu") (hatch edge 0.508)
+    (connect_pads thru_hole_only (clearance 0.3))
+    (fill yes (thermal_gap 0.508) (thermal_bridge_width 0.508))
+    (polygon
+      (pts
+        (xy 80 0)
+        (xy 168 0)
+        (xy 168 100)
+        (xy 80 100)
+      )
     )
   )
