File: LightRail_LPO_1.6T.kicad_pcb (KiCad board)
At the start: 10 copper layers, 168 x 105 mm, 234 parts, among them J1 MPO-24, U1 TFLN_Mod_Gen3_8CH, U101 AI_SoC_U0, U102 TFLN_PIC_U0, U2 NeoPhotonics_1550nm_DFB, U201 AI_SoC_U1, U202 TFLN_PIC_U1, U3 Si5395A, U302 ISL99390, U303 ISL99390, U304 ISL99390, U305 ISL99390, U306 ISL99390, U307 ISL99390, U326 ISL99390, U327 ISL99390, U328 ISL99390, U329 ISL99390, U330 ISL99390, U331 ISL99390, U4 AD5684R, U5 MAX3669, U6 TPS7A2018, U7 TPS54360, U8 MPT5000

Commit message: feat: HBM4 co-packaged memory migration (DDR5 -> HBM4 interposer)
Replace discrete DDR5-8800 DIMM fly-by subsystem with a co-packaged
NCE+HBM4-on-interposer topology per vendor reference (SK hynix /
Micron 12-Hi, 48 GB/stack, 8 Gbps/pin, 1024-bit bus).

PCB (LightRail_LPO_1.6T.kicad_pcb):
- Remove 8x DDR5 DIMM footprints (U202/U204/U206/U208 + U2102/..)
- Add 8x HBM4_Stack_11x11mm footprints (U103-U106 flanking U101,
  U203-U206 flanking U201) sitting on the co-packaged interposer
- Remove DDR5 CK fly-by segments on In2.Cu; nets 148-163 renamed
  DDR5_U{0,1}_* -> HBM4_U{0,1}_* (VDDC_S/VDDQL_S/VDDQ_S/VPP_S,
  REFCK_P/N, CATTRIP, PWR_GOOD, TCK/TMS/TDI/TDO)
- Silk text relabelled: 'DDR5-8800 Memory Bus (Fly-by Topology)'
  -> 'HBM4 Co-Packaged Memory (Advanced Interposer Path)'; central
  BGA value 'AI Compute Units (TFLN Photonics Enabled, NCE+HBM4
  Stack)'; bottom caption 'NCE+HBM4 Co-Packaged TFLN Photonics-
  integrated AI Compute Node (Based on MBoard [with 8x PCIe 5.0
  Slots])'
- Silicon interposer courtyard outlines added on F.Fab around each
  NCE+HBM4 module

Schematic:
- Memory.kicad_sch rewritten as HBM4_Stack_12Hi template (9 external
  side-channel pins + IEEE-1500 test bus)
- LightRail_LPO_1.6T.kicad_sch: 32 MEM_U*_D* DIMM sheets dropped;
  8 HBM4 stack sheets added; DDR5A_* sheet pins renamed HBM4_* on
  both AI_Core_Unit instances
- AI_Core.kicad_sch: DDR5A_* port names renamed HBM4_*
- .kicad_pro: net class DDR5_Data -> HBM4_Interposer

Fab:
- drc_custom.kicad_dru rewritten for HBM4 side-channel (REFCK 100 Ohm
  diff, IEEE-1500 50 Ohm SE, length 5-35 mm, P/N match +/-0.025 mm)
- generate_bom.py: 32 DDR5 DIMM entries -> 8 HBM4 stacks (SK hynix
  H56G48AT5DX117, marked 'TP' / DNP as vendor-supplied); VDDQ buck
  redescribed for HBM4; BOM.csv / BOM.md regenerated
- generate_pinouts.py: pinout_DDR5_DIMM.csv -> pinout_HBM4_Stack.csv;
  SoC BGA-2500 pinout table now lists VDDC/VDDQL/VDDQ/VPP HBM4 domains
  and flags the 1024x4 data bus as INTERPOSER-INTERN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
Parts:
- added U103: HBM4_12Hi_48GB, LightRail:HBM4_Stack_11x11mm, F.Cu at (16.0, 40.0)
- added U104: HBM4_12Hi_48GB, LightRail:HBM4_Stack_11x11mm, F.Cu at (16.0, 60.0)
- added U105: HBM4_12Hi_48GB, LightRail:HBM4_Stack_11x11mm, F.Cu at (68.0, 40.0)
- added U106: HBM4_12Hi_48GB, LightRail:HBM4_Stack_11x11mm, F.Cu at (68.0, 60.0)
- added U203: HBM4_12Hi_48GB, LightRail:HBM4_Stack_11x11mm, F.Cu at (100.0, 40.0)
- added U204: HBM4_12Hi_48GB, LightRail:HBM4_Stack_11x11mm, F.Cu at (100.0, 60.0)
- added U205: HBM4_12Hi_48GB, LightRail:HBM4_Stack_11x11mm, F.Cu at (152.0, 40.0)
- added U206: HBM4_12Hi_48GB, LightRail:HBM4_Stack_11x11mm, F.Cu at (152.0, 60.0)
Routing:
- net DDR5_U1_CK_P: track 59.0 -> 0.00 mm
- net DDR5_U1_CK_N: track 59.0 -> 0.00 mm
- net DDR5_U0_CK_P: track 59.0 -> 0.00 mm
- net DDR5_U0_CK_N: track 59.0 -> 0.00 mm
Other:
- board text added: "AI COMPUTE UNIT 0 (TFLN Photonics Enabled, NCE+HBM4 Stack)"
- board text added: "AI COMPUTE UNIT 1 (TFLN Photonics Enabled, NCE+HBM4 Stack)"
- board text added: "HBM4 CO-PACKAGED MEMORY (Advanced Interposer Path)"
- board text added: "LightRail LPO 1.6T NCE+HBM4 Co-Packaged TFLN Photonics-integrated AI Compute Node (Based on MBoard [with 8x PCIe 5.0 Slots]) Rev 4.0"
- board text added: "SILICON INTERPOSER (NCE+4xHBM4)"
- board text removed: "AI COMPUTE UNIT 0"
- board text removed: "AI COMPUTE UNIT 1"
- board text removed: "DDR5 DIMM SLOTS"
- board text removed: "LightRail LPO 1.6T Dual AI Compute Node Rev 4.0"
