File: AI_Core.kicad_sch (KiCad schematic)
At the start: 9 parts, among them U101 AI_SoC_BGA_2500

Commit message: fix: DDR5 DQS0 naming consistency + gerber X2 flag
- export_gerbers.sh: drop --no-x2 so X2 extended attributes are emitted
  (matches docs which advertise RS-274X/X2 to the fab)
- Root schematic sheet pins DDR5A_DQS0_P/_N -> DDR5A_DQS0P/N on both
  AI_Core_Unit0 and AI_Core_Unit1 to match the SoC symbol pin names
- Add matching hierarchical_label 'DDR5A_DQS0P' / 'DDR5A_DQS0N' in
  AI_Core.kicad_sch so the DQS0 strobe is actually wired through the
  hierarchy (DQS1-3 remain on the residual-items list)

Co-Authored-By: Bola Olatunji <bola.olatunji@ai.lightos.sh>
Changed lines of the file:
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@@
   (hierarchical_label "I2C_SDA" (shape bidirectional) (at 40.64 76.0 180) (effects (font (size 1.27 1.27))))
   (hierarchical_label "I2C_SCL" (shape input) (at 40.64 79.0 180) (effects (font (size 1.27 1.27))))
+  (hierarchical_label "DDR5A_DQS0P" (shape bidirectional) (at 264.16 120.47 0) (effects (font (size 1.27 1.27))))
+  (hierarchical_label "DDR5A_DQS0N" (shape bidirectional) (at 264.16 119.20 0) (effects (font (size 1.27 1.27))))
   (text "AI COMPUTE UNIT - CORE\nAI SoC BGA: 2500 pins, 0.8mm pitch\nTFLN Photonic Engine Interface: 8ch RF differential\nDDR5 Memory Controller: Channel A (32-bit + ECC)\nPCIe Gen 6.0 x16: 64 GT/s per lane\nV_core: 0.8V, 1000A (24-phase DrMOS)" (at 152.4 30.48 0) (effects (font (size 2.0 2.0)) (justify left)))
 ) ;; end kicad_sch

Commit message: fix(sch): add VDDQ hierarchical pin/label on AI_Core; README residual items
Devin Review flagged two doc/schematic gaps:

1. AI SoC VDDQ (DDR5 PHY I/O supply, 1.1 V) had a power_in pin on the
   AI_SoC symbol in AI_Core.kicad_sch but no hierarchical_label and no
   matching sheet pin on either AI_Core_Unit instance in the root
   schematic, so the rail was dangling at the hierarchy boundary. The
   VDDQ regulator (U31, TPS544C20) could not supply the SoC through the
   interface.

2. README residual items section still listed VDD_IO, TFLN_CLK_P/N, and
   VRM VID0/1/2 as missing -- these were added in Rev 4.1 and are
   already present, so the stale list would mislead the next engineer
   into adding duplicates and would hide the real missing pin (VDDQ).

Fixes: - Add hierarchical_label "VDDQ" (shape input) to AI_Core.kicad_sch
    alongside V_CORE and VDD_IO.
  - Add (pin "VDDQ" input ...) on both AI_Core_Unit0 and
    AI_Core_Unit1 sheet instances in LightRail_LPO_1.6T.kicad_sch,
    slotted between VDD_IO and TFLN_CLK_P with a 0.63 mm offset.
  - Rewrite README residual items to list only the genuinely missing
    DDR5 lane pins (DQ8..31, DQS1..3, DM1..3, CA4..13, CS1) and
    explicitly note that VDD_IO / VDDQ / TFLN_CLK / VID0..2 are done.
  - Add Rev 4.2 row to the revision history summarizing all the
    parse-fix / export / DRC / BOM fixes from this session.
Co-Authored-By: Bola Olatunji <bola.olatunji@ai.lightos.sh>
Changed lines of the file:
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@@
   (hierarchical_label "V_CORE" (shape input) (at 40.64 60.0 180) (effects (font (size 1.27 1.27))))
   (hierarchical_label "VDD_IO" (shape input) (at 40.64 63.0 180) (effects (font (size 1.27 1.27))))
+  (hierarchical_label "VDDQ" (shape input) (at 40.64 64.5 180) (effects (font (size 1.27 1.27))))
   (hierarchical_label "GND" (shape passive) (at 40.64 66.0 180) (effects (font (size 1.27 1.27))))
   (hierarchical_label "TFLN_CLK_P" (shape output) (at 40.64 70.0 180) (effects (font (size 1.27 1.27))))
