File: AI_Core.kicad_sch (KiCad schematic)
At the start: 9 parts, among them U101 AI_SoC_BGA_2500

Commit message: feat: HBM4 co-packaged memory migration (DDR5 -> HBM4 interposer)
Replace discrete DDR5-8800 DIMM fly-by subsystem with a co-packaged
NCE+HBM4-on-interposer topology per vendor reference (SK hynix /
Micron 12-Hi, 48 GB/stack, 8 Gbps/pin, 1024-bit bus).

PCB (LightRail_LPO_1.6T.kicad_pcb):
- Remove 8x DDR5 DIMM footprints (U202/U204/U206/U208 + U2102/..)
- Add 8x HBM4_Stack_11x11mm footprints (U103-U106 flanking U101,
  U203-U206 flanking U201) sitting on the co-packaged interposer
- Remove DDR5 CK fly-by segments on In2.Cu; nets 148-163 renamed
  DDR5_U{0,1}_* -> HBM4_U{0,1}_* (VDDC_S/VDDQL_S/VDDQ_S/VPP_S,
  REFCK_P/N, CATTRIP, PWR_GOOD, TCK/TMS/TDI/TDO)
- Silk text relabelled: 'DDR5-8800 Memory Bus (Fly-by Topology)'
  -> 'HBM4 Co-Packaged Memory (Advanced Interposer Path)'; central
  BGA value 'AI Compute Units (TFLN Photonics Enabled, NCE+HBM4
  Stack)'; bottom caption 'NCE+HBM4 Co-Packaged TFLN Photonics-
  integrated AI Compute Node (Based on MBoard [with 8x PCIe 5.0
  Slots])'
- Silicon interposer courtyard outlines added on F.Fab around each
  NCE+HBM4 module

Schematic:
- Memory.kicad_sch rewritten as HBM4_Stack_12Hi template (9 external
  side-channel pins + IEEE-1500 test bus)
- LightRail_LPO_1.6T.kicad_sch: 32 MEM_U*_D* DIMM sheets dropped;
  8 HBM4 stack sheets added; DDR5A_* sheet pins renamed HBM4_* on
  both AI_Core_Unit instances
- AI_Core.kicad_sch: DDR5A_* port names renamed HBM4_*
- .kicad_pro: net class DDR5_Data -> HBM4_Interposer

Fab:
- drc_custom.kicad_dru rewritten for HBM4 side-channel (REFCK 100 Ohm
  diff, IEEE-1500 50 Ohm SE, length 5-35 mm, P/N match +/-0.025 mm)
- generate_bom.py: 32 DDR5 DIMM entries -> 8 HBM4 stacks (SK hynix
  H56G48AT5DX117, marked 'TP' / DNP as vendor-supplied); VDDQ buck
  redescribed for HBM4; BOM.csv / BOM.md regenerated
- generate_pinouts.py: pinout_DDR5_DIMM.csv -> pinout_HBM4_Stack.csv;
  SoC BGA-2500 pinout table now lists VDDC/VDDQL/VDDQ/VPP HBM4 domains
  and flags the 1024x4 data bus as INTERPOSER-INTERN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
Other:
- note added: "AI COMPUTE UNIT - CORE (NCE + 4x HBM4 stacks, co-packaged) NCE BGA: 2500 pins, 0.8mm pitch (composite module: NCE die + silicon interposer + 4x HBM4 12-Hi) TFLN Photonic Engine Interface: 8ch RF differential HBM4 Memory: 4 stacks × 1024 lanes @ 8 Gbps/pin (interposer-internal) PCIe Gen 6.0 x16: 64 GT/s per lane V_core: 0.8V, 1000A+ (24-phase DrMOS, NCE + HBM4 combined load)"
- note removed: "AI COMPUTE UNIT - CORE AI SoC BGA: 2500 pins, 0.8mm pitch TFLN Photonic Engine Interface: 8ch RF differential DDR5 Memory Controller: Channel A (32-bit + ECC) PCIe Gen 6.0 x16: 64 GT/s per lane V_core: 0.8V, 1000A (24-phase DrMOS)"
