File: LightRail_LPO_1.6T.kicad_sch (KiCad schematic)
At the start: 9 parts, among them J1 MPO-24, U1 TFLN_Mod_Gen3_8CH, U2 NeoPhotonics_1550nm_DFB, U3 Si5395A, U4 AD5684R, U5 MAX3669, U6 TPS7A2018, U7 TPS54360, U8 MPT5000

Commit message: feat: implement dual AI Compute Node with TFLN photonic integration
- Add hierarchical sub-sheets: AI_Core (SoC BGA 2500-pin, TFLN interface),
  Memory (DDR5 DIMM 288-pin fly-by topology), VRM (24-phase DrMOS array)
- Update root schematic with dual compute unit hierarchy (2x AI_Core,
  2x VRM, 32x Memory sheets)
- Add net classes: TFLN_RF (0.15mm/0.20mm diff), PCIe_Gen6 (0.12mm/0.18mm),
  DDR5_Data (0.10mm/0.15mm micro-via), PWR_CORE (2.0mm+)
- Create custom footprints: BGA-2500 (50x50, 0.8mm pitch), TFLN_PIC
  (periphery pads, optical keepout center), DrMOS PowerPAK 8x8mm,
  DDR5 DIMM 288-pin connector
- Update PCB: TFLN keepout zones, VRM V_core copper pours on internal
  layers, GND reference plane, DDR5 fly-by routing structures
- Place AI SoC BGA, TFLN PIC, and DrMOS footprints for both units
- Update project rev to 4.0, date to 2026-04-11

Co-Authored-By: Bola Olatunji <bola.olatunji@ai.lightos.sh>
Other:
- added sheet AI_Core_Unit0 (AI_Core.kicad_sch)
- added sheet AI_Core_Unit1 (AI_Core.kicad_sch)
- added sheet MEM_U0_D0 (Memory.kicad_sch)
- added sheet MEM_U0_D1 (Memory.kicad_sch)
- added sheet MEM_U0_D10 (Memory.kicad_sch)
- added sheet MEM_U0_D11 (Memory.kicad_sch)
- added sheet MEM_U0_D12 (Memory.kicad_sch)
- added sheet MEM_U0_D13 (Memory.kicad_sch)
- added sheet MEM_U0_D14 (Memory.kicad_sch)
- added sheet MEM_U0_D15 (Memory.kicad_sch)
- added sheet MEM_U0_D2 (Memory.kicad_sch)
- added sheet MEM_U0_D3 (Memory.kicad_sch)
- added sheet MEM_U0_D4 (Memory.kicad_sch)
- added sheet MEM_U0_D5 (Memory.kicad_sch)
- added sheet MEM_U0_D6 (Memory.kicad_sch)
- added sheet MEM_U0_D7 (Memory.kicad_sch)
- added sheet MEM_U0_D8 (Memory.kicad_sch)
- added sheet MEM_U0_D9 (Memory.kicad_sch)
- added sheet MEM_U1_D0 (Memory.kicad_sch)
- added sheet MEM_U1_D1 (Memory.kicad_sch)
- added sheet MEM_U1_D10 (Memory.kicad_sch)
- added sheet MEM_U1_D11 (Memory.kicad_sch)
- added sheet MEM_U1_D12 (Memory.kicad_sch)
- added sheet MEM_U1_D13 (Memory.kicad_sch)
- added sheet MEM_U1_D14 (Memory.kicad_sch)
- added sheet MEM_U1_D15 (Memory.kicad_sch)
- added sheet MEM_U1_D2 (Memory.kicad_sch)
- added sheet MEM_U1_D3 (Memory.kicad_sch)
- added sheet MEM_U1_D4 (Memory.kicad_sch)
- added sheet MEM_U1_D5 (Memory.kicad_sch)
- added sheet MEM_U1_D6 (Memory.kicad_sch)
- added sheet MEM_U1_D7 (Memory.kicad_sch)
- added sheet MEM_U1_D8 (Memory.kicad_sch)
- added sheet MEM_U1_D9 (Memory.kicad_sch)
- added sheet VRM_Unit0 (VRM.kicad_sch)
- added sheet VRM_Unit1 (VRM.kicad_sch)
- note added: "DUAL AI COMPUTE UNITS Each unit: AI SoC BGA (2500 pins) + 16x DDR5 DIMMs + 24-phase VRM TFLN Photonic Engine: 8ch RF differential per unit Total: 1.6 Tbps aggregate optical bandwidth PCIe Gen6 x16 per unit (64 GT/s per lane) V_core: 0.8V, 1000A per unit (24-phase DrMOS)"

Commit message: fix: add missing VDD_IO, TFLN_CLK, DDR5, and VID pins to sheet instances
- AI_Core_Unit0/Unit1: add VDD_IO (I/O power rail), TFLN_CLK_P/N (photonic
  engine clock), DDR5A_CK_P/N, CS0, CA0-CA3, DQ0-DQ7, DQS0_P/N (memory
  controller interface)
- VRM_Unit0/Unit1: add VID0/VID1/VID2 (voltage ID programming for ISL69260)

Co-Authored-By: Bola Olatunji <bola.olatunji@ai.lightos.sh>
Other:
- sheet AI_Core_Unit0 ports: added DDR5A_CA0, DDR5A_CA1, DDR5A_CA2, DDR5A_CA3, DDR5A_CK_N, DDR5A_CK_P, DDR5A_CS0, DDR5A_DQ0, DDR5A_DQ1, DDR5A_DQ2, DDR5A_DQ3, DDR5A_DQ4, DDR5A_DQ5, DDR5A_DQ6, DDR5A_DQ7, DDR5A_DQS0_N, DDR5A_DQS0_P, TFLN_CLK_N, TFLN_CLK_P, VDD_IO; removed none
- sheet AI_Core_Unit1 ports: added DDR5A_CA0, DDR5A_CA1, DDR5A_CA2, DDR5A_CA3, DDR5A_CK_N, DDR5A_CK_P, DDR5A_CS0, DDR5A_DQ0, DDR5A_DQ1, DDR5A_DQ2, DDR5A_DQ3, DDR5A_DQ4, DDR5A_DQ5, DDR5A_DQ6, DDR5A_DQ7, DDR5A_DQS0_N, DDR5A_DQS0_P, TFLN_CLK_N, TFLN_CLK_P, VDD_IO; removed none
- sheet VRM_Unit0 ports: added VID0, VID1, VID2; removed none
- sheet VRM_Unit1 ports: added VID0, VID1, VID2; removed none
Changed lines of the file:
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@@
     (pin "PCIE_TX15P" bidirectional (at 110.8 294.05 0) (effects (font (size 1.0 1.0))))
     (pin "PCIE_TX15N" bidirectional (at 110.8 294.68 0) (effects (font (size 1.0 1.0))))
+    (pin "VDD_IO" input (at 50.8 300.40 180) (effects (font (size 1.0 1.0))))
+    (pin "TFLN_CLK_P" output (at 50.8 301.67 180) (effects (font (size 1.0 1.0))))
+    (pin "TFLN_CLK_N" output (at 50.8 302.94 180) (effects (font (size 1.0 1.0))))
+    (pin "DDR5A_CK_P" output (at 110.8 296.00 0) (effects (font (size 1.0 1.0))))
+    (pin "DDR5A_CK_N" output (at 110.8 296.63 0) (effects (font (size 1.0 1.0))))
+    (pin "DDR5A_CS0" output (at 110.8 297.27 0) (effects (font (size 1.0 1.0))))
+    (pin "DDR5A_CA0" output (at 110.8 297.90 0) (effects (font (size 1.0 1.0))))
+    (pin "DDR5A_CA1" output (at 110.8 298.54 0) (effects (font (size 1.0 1.0))))
+    (pin "DDR5A_CA2" output (at 110.8 299.17 0) (effects (font (size 1.0 1.0))))
+    (pin "DDR5A_CA3" output (at 110.8 299.81 0) (effects (font (size 1.0 1.0))))
+    (pin "DDR5A_DQ0" bidirectional (at 110.8 300.44 0) (effects (font (size 1.0 1.0))))
+    (pin "DDR5A_DQ1" bidirectional (at 110.8 301.08 0) (effects (font (size 1.0 1.0))))
+    (pin "DDR5A_DQ2" bidirectional (at 110.8 301.71 0) (effects (font (size 1.0 1.0))))
+    (pin "DDR5A_DQ3" bidirectional (at 110.8 302.35 0) (effects (font (size 1.0 1.0))))
+    (pin "DDR5A_DQ4" bidirectional (at 110.8 302.98 0) (effects (font (size 1.0 1.0))))
+    (pin "DDR5A_DQ5" bidirectional (at 110.8 303.62 0) (effects (font (size 1.0 1.0))))
+    (pin "DDR5A_DQ6" bidirectional (at 110.8 304.25 0) (effects (font (size 1.0 1.0))))
+    (pin "DDR5A_DQ7" bidirectional (at 110.8 304.89 0) (effects (font (size 1.0 1.0))))
+    (pin "DDR5A_DQS0_P" bidirectional (at 110.8 305.52 0) (effects (font (size 1.0 1.0))))
+    (pin "DDR5A_DQS0_N" bidirectional (at 110.8 306.16 0) (effects (font (size 1.0 1.0))))
   )
   (sheet (at 200.0 270.0) (size 60.0 40.0)
@@
     (pin "PCIE_TX15P" bidirectional (at 260.0 294.05 0) (effects (font (size 1.0 1.0))))
     (pin "PCIE_TX15N" bidirectional (at 260.0 294.68 0) (effects (font (size 1.0 1.0))))
+    (pin "VDD_IO" input (at 200.0 300.40 180) (effects (font (size 1.0 1.0))))
+    (pin "TFLN_CLK_P" output (at 200.0 301.67 180) (effects (font (size 1.0 1.0))))
+    (pin "TFLN_CLK_N" output (at 200.0 302.94 180) (effects (font (size 1.0 1.0))))
+    (pin "DDR5A_CK_P" output (at 260.0 296.00 0) (effects (font (size 1.0 1.0))))
+    (pin "DDR5A_CK_N" output (at 260.0 296.63 0) (effects (font (size 1.0 1.0))))
+    (pin "DDR5A_CS0" output (at 260.0 297.27 0) (effects (font (size 1.0 1.0))))
+    (pin "DDR5A_CA0" output (at 260.0 297.90 0) (effects (font (size 1.0 1.0))))
+    (pin "DDR5A_CA1" output (at 260.0 298.54 0) (effects (font (size 1.0 1.0))))
+    (pin "DDR5A_CA2" output (at 260.0 299.17 0) (effects (font (size 1.0 1.0))))
+    (pin "DDR5A_CA3" output (at 260.0 299.81 0) (effects (font (size 1.0 1.0))))
+    (pin "DDR5A_DQ0" bidirectional (at 260.0 300.44 0) (effects (font (size 1.0 1.0))))
+    (pin "DDR5A_DQ1" bidirectional (at 260.0 301.08 0) (effects (font (size 1.0 1.0))))
+    (pin "DDR5A_DQ2" bidirectional (at 260.0 301.71 0) (effects (font (size 1.0 1.0))))
+    (pin "DDR5A_DQ3" bidirectional (at 260.0 302.35 0) (effects (font (size 1.0 1.0))))
+    (pin "DDR5A_DQ4" bidirectional (at 260.0 302.98 0) (effects (font (size 1.0 1.0))))
+    (pin "DDR5A_DQ5" bidirectional (at 260.0 303.62 0) (effects (font (size 1.0 1.0))))
+    (pin "DDR5A_DQ6" bidirectional (at 260.0 304.25 0) (effects (font (size 1.0 1.0))))
+    (pin "DDR5A_DQ7" bidirectional (at 260.0 304.89 0) (effects (font (size 1.0 1.0))))
+    (pin "DDR5A_DQS0_P" bidirectional (at 260.0 305.52 0) (effects (font (size 1.0 1.0))))
+    (pin "DDR5A_DQS0_N" bidirectional (at 260.0 306.16 0) (effects (font (size 1.0 1.0))))
   )
   (sheet (at 50.8 320.0) (size 60.0 25.0)
@@
     (pin "I2C_SCL" input (at 50.8 334.0 180) (effects (font (size 1.0 1.0))))
     (pin "EN" input (at 50.8 337.0 180) (effects (font (size 1.0 1.0))))
+    (pin "VID0" input (at 50.8 340.0 180) (effects (font (size 1.0 1.0))))
+    (pin "VID1" input (at 50.8 341.5 180) (effects (font (size 1.0 1.0))))
+    (pin "VID2" input (at 50.8 343.0 180) (effects (font (size 1.0 1.0))))
   )
   (sheet (at 200.0 320.0) (size 60.0 25.0)
@@
     (pin "I2C_SCL" input (at 200.0 334.0 180) (effects (font (size 1.0 1.0))))
     (pin "EN" input (at 200.0 337.0 180) (effects (font (size 1.0 1.0))))
+    (pin "VID0" input (at 200.0 340.0 180) (effects (font (size 1.0 1.0))))
+    (pin "VID1" input (at 200.0 341.5 180) (effects (font (size 1.0 1.0))))
+    (pin "VID2" input (at 200.0 343.0 180) (effects (font (size 1.0 1.0))))
   )
   (sheet (at 50.8 355.0) (size 12.0 15.0)

Commit message: fix: DDR5 DQS0 naming consistency + gerber X2 flag
- export_gerbers.sh: drop --no-x2 so X2 extended attributes are emitted
  (matches docs which advertise RS-274X/X2 to the fab)
- Root schematic sheet pins DDR5A_DQS0_P/_N -> DDR5A_DQS0P/N on both
  AI_Core_Unit0 and AI_Core_Unit1 to match the SoC symbol pin names
- Add matching hierarchical_label 'DDR5A_DQS0P' / 'DDR5A_DQS0N' in
  AI_Core.kicad_sch so the DQS0 strobe is actually wired through the
  hierarchy (DQS1-3 remain on the residual-items list)

Co-Authored-By: Bola Olatunji <bola.olatunji@ai.lightos.sh>
Other:
- sheet AI_Core_Unit1 ports: added DDR5A_DQS0N, DDR5A_DQS0P; removed DDR5A_DQS0_N, DDR5A_DQS0_P
Changed lines of the file:
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@@
     (pin "DDR5A_DQ6" bidirectional (at 260.0 304.25 0) (effects (font (size 1.0 1.0))))
     (pin "DDR5A_DQ7" bidirectional (at 260.0 304.89 0) (effects (font (size 1.0 1.0))))
-    (pin "DDR5A_DQS0_P" bidirectional (at 260.0 305.52 0) (effects (font (size 1.0 1.0))))
-    (pin "DDR5A_DQS0_N" bidirectional (at 260.0 306.16 0) (effects (font (size 1.0 1.0))))
+    (pin "DDR5A_DQS0P" bidirectional (at 260.0 305.52 0) (effects (font (size 1.0 1.0))))
+    (pin "DDR5A_DQS0N" bidirectional (at 260.0 306.16 0) (effects (font (size 1.0 1.0))))
   )
   (sheet (at 50.8 320.0) (size 60.0 25.0)

Commit message: fix: DDR5A_DQS0 sheet pins on AI_Core_Unit0 (previous commit only caught Unit1)
Rename pin DDR5A_DQS0_P -> DDR5A_DQS0P and DDR5A_DQS0_N -> DDR5A_DQS0N
on the AI_Core_Unit0 sheet instance (lines 580-581) to match the
already-fixed Unit1 instance, the SoC symbol pins in AI_Core.kicad_sch
lines 105-106, and the hierarchical labels in AI_Core.kicad_sch lines
337-338.

Co-Authored-By: Bola Olatunji <bola.olatunji@ai.lightos.sh>
Other:
- sheet AI_Core_Unit0 ports: added DDR5A_DQS0N, DDR5A_DQS0P; removed DDR5A_DQS0_N, DDR5A_DQS0_P
Changed lines of the file:
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@@
     (pin "DDR5A_DQ6" bidirectional (at 110.8 304.25 0) (effects (font (size 1.0 1.0))))
     (pin "DDR5A_DQ7" bidirectional (at 110.8 304.89 0) (effects (font (size 1.0 1.0))))
-    (pin "DDR5A_DQS0_P" bidirectional (at 110.8 305.52 0) (effects (font (size 1.0 1.0))))
-    (pin "DDR5A_DQS0_N" bidirectional (at 110.8 306.16 0) (effects (font (size 1.0 1.0))))
+    (pin "DDR5A_DQS0P" bidirectional (at 110.8 305.52 0) (effects (font (size 1.0 1.0))))
+    (pin "DDR5A_DQS0N" bidirectional (at 110.8 306.16 0) (effects (font (size 1.0 1.0))))
   )
   (sheet (at 200.0 270.0) (size 60.0 40.0)

Commit message: fix(pcb,sch,drc): make files kicad-cli-parseable + VDDQ + DRC regex
Net result: 'kicad-cli pcb export gerbers' now successfully produces a
full fab package (gerbers/, drill/, assembly/, docs/) from the scaffold.

PCB edits (needed for kicad-cli to parse):
- Strip top-level ';; comment' lines from .kicad_pcb (KiCad S-expr
  parser rejects them outside of whitespace positions)
- Remove '(id N)' tokens from footprint 'property' blocks (that form
  is schematic-only; in .kicad_pcb it is not an allowed token)

Schematic edits:
- Add VDDQ hierarchical sheet-pin to all 32 Memory sheet instances so
  the DDR5 1.1V data-I/O rail actually propagates through hierarchy

DRC edits:
- The DDR5_CK / DDR5_CA net classes don't exist in the project — only
  DDR5_Data does. Rewrite ddr5_ck_ca_length_match condition to match
  DDR5_Data nets whose names look like *_CK_P/N, *_CA<n>, *_CS<n> via
  regex so the skew rule actually fires.

Co-Authored-By: Bola Olatunji <bola.olatunji@ai.lightos.sh>
Other:
- sheet MEM_U0_D0 ports: added VDDQ; removed none
- sheet MEM_U0_D1 ports: added VDDQ; removed none
- sheet MEM_U0_D10 ports: added VDDQ; removed none
- sheet MEM_U0_D11 ports: added VDDQ; removed none
- sheet MEM_U0_D12 ports: added VDDQ; removed none
- sheet MEM_U0_D13 ports: added VDDQ; removed none
- sheet MEM_U0_D14 ports: added VDDQ; removed none
- sheet MEM_U0_D15 ports: added VDDQ; removed none
- sheet MEM_U0_D2 ports: added VDDQ; removed none
- sheet MEM_U0_D3 ports: added VDDQ; removed none
- sheet MEM_U0_D4 ports: added VDDQ; removed none
- sheet MEM_U0_D5 ports: added VDDQ; removed none
- sheet MEM_U0_D6 ports: added VDDQ; removed none
- sheet MEM_U0_D7 ports: added VDDQ; removed none
- sheet MEM_U0_D8 ports: added VDDQ; removed none
- sheet MEM_U0_D9 ports: added VDDQ; removed none
- sheet MEM_U1_D0 ports: added VDDQ; removed none
- sheet MEM_U1_D1 ports: added VDDQ; removed none
- sheet MEM_U1_D10 ports: added VDDQ; removed none
- sheet MEM_U1_D11 ports: added VDDQ; removed none
- sheet MEM_U1_D12 ports: added VDDQ; removed none
- sheet MEM_U1_D13 ports: added VDDQ; removed none
- sheet MEM_U1_D14 ports: added VDDQ; removed none
- sheet MEM_U1_D15 ports: added VDDQ; removed none
- sheet MEM_U1_D2 ports: added VDDQ; removed none
- sheet MEM_U1_D3 ports: added VDDQ; removed none
- sheet MEM_U1_D4 ports: added VDDQ; removed none
- sheet MEM_U1_D5 ports: added VDDQ; removed none
- sheet MEM_U1_D6 ports: added VDDQ; removed none
- sheet MEM_U1_D7 ports: added VDDQ; removed none
- sheet MEM_U1_D8 ports: added VDDQ; removed none
- sheet MEM_U1_D9 ports: added VDDQ; removed none
Changed lines of the file:
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@@
     (pin "VDD" input (at 62.8 358.0 0) (effects (font (size 0.8 0.8))))
     (pin "VSS" passive (at 62.8 359.5 0) (effects (font (size 0.8 0.8))))
+    (pin "VDDQ" input (at 62.8 361.0 0) (effects (font (size 0.8 0.8))))
   )
   (sheet (at 65.8 355.0) (size 12.0 15.0)
@@
     (pin "VDD" input (at 77.8 358.0 0) (effects (font (size 0.8 0.8))))
     (pin "VSS" passive (at 77.8 359.5 0) (effects (font (size 0.8 0.8))))
+    (pin "VDDQ" input (at 77.8 361.0 0) (effects (font (size 0.8 0.8))))
   )
   (sheet (at 80.8 355.0) (size 12.0 15.0)
@@
     (pin "VDD" input (at 92.8 358.0 0) (effects (font (size 0.8 0.8))))
     (pin "VSS" passive (at 92.8 359.5 0) (effects (font (size 0.8 0.8))))
+    (pin "VDDQ" input (at 92.8 361.0 0) (effects (font (size 0.8 0.8))))
   )
   (sheet (at 95.8 355.0) (size 12.0 15.0)
@@
     (pin "VDD" input (at 107.8 358.0 0) (effects (font (size 0.8 0.8))))
     (pin "VSS" passive (at 107.8 359.5 0) (effects (font (size 0.8 0.8))))
+    (pin "VDDQ" input (at 107.8 361.0 0) (effects (font (size 0.8 0.8))))
   )
   (sheet (at 50.8 375.0) (size 12.0 15.0)
@@
     (pin "VDD" input (at 62.8 378.0 0) (effects (font (size 0.8 0.8))))
     (pin "VSS" passive (at 62.8 379.5 0) (effects (font (size 0.8 0.8))))
+    (pin "VDDQ" input (at 62.8 381.0 0) (effects (font (size 0.8 0.8))))
   )
   (sheet (at 65.8 375.0) (size 12.0 15.0)
@@
     (pin "VDD" input (at 77.8 378.0 0) (effects (font (size 0.8 0.8))))
     (pin "VSS" passive (at 77.8 379.5 0) (effects (font (size 0.8 0.8))))
+    (pin "VDDQ" input (at 77.8 381.0 0) (effects (font (size 0.8 0.8))))
   )
   (sheet (at 80.8 375.0) (size 12.0 15.0)
@@
     (pin "VDD" input (at 92.8 378.0 0) (effects (font (size 0.8 0.8))))
     (pin "VSS" passive (at 92.8 379.5 0) (effects (font (size 0.8 0.8))))
+    (pin "VDDQ" input (at 92.8 381.0 0) (effects (font (size 0.8 0.8))))
   )
   (sheet (at 95.8 375.0) (size 12.0 15.0)
@@
     (pin "VDD" input (at 107.8 378.0 0) (effects (font (size 0.8 0.8))))
     (pin "VSS" passive (at 107.8 379.5 0) (effects (font (size 0.8 0.8))))
+    (pin "VDDQ" input (at 107.8 381.0 0) (effects (font (size 0.8 0.8))))
   )
   (sheet (at 50.8 395.0) (size 12.0 15.0)
@@
     (pin "VDD" input (at 62.8 398.0 0) (effects (font (size 0.8 0.8))))
     (pin "VSS" passive (at 62.8 399.5 0) (effects (font (size 0.8 0.8))))
+    (pin "VDDQ" input (at 62.8 401.0 0) (effects (font (size 0.8 0.8))))
   )
   (sheet (at 65.8 395.0) (size 12.0 15.0)
@@
     (pin "VDD" input (at 77.8 398.0 0) (effects (font (size 0.8 0.8))))
     (pin "VSS" passive (at 77.8 399.5 0) (effects (font (size 0.8 0.8))))
+    (pin "VDDQ" input (at 77.8 401.0 0) (effects (font (size 0.8 0.8))))
   )
   (sheet (at 80.8 395.0) (size 12.0 15.0)
@@
     (pin "VDD" input (at 92.8 398.0 0) (effects (font (size 0.8 0.8))))
     (pin "VSS" passive (at 92.8 399.5 0) (effects (font (size 0.8 0.8))))
+    (pin "VDDQ" input (at 92.8 401.0 0) (effects (font (size 0.8 0.8))))
   )
   (sheet (at 95.8 395.0) (size 12.0 15.0)
@@
     (pin "VDD" input (at 107.8 398.0 0) (effects (font (size 0.8 0.8))))
     (pin "VSS" passive (at 107.8 399.5 0) (effects (font (size 0.8 0.8))))
+    (pin "VDDQ" input (at 107.8 401.0 0) (effects (font (size 0.8 0.8))))
   )
   (sheet (at 50.8 415.0) (size 12.0 15.0)
@@
     (pin "VDD" input (at 62.8 418.0 0) (effects (font (size 0.8 0.8))))
     (pin "VSS" passive (at 62.8 419.5 0) (effects (font (size 0.8 0.8))))
+    (pin "VDDQ" input (at 62.8 421.0 0) (effects (font (size 0.8 0.8))))
   )
   (sheet (at 65.8 415.0) (size 12.0 15.0)
@@
     (pin "VDD" input (at 77.8 418.0 0) (effects (font (size 0.8 0.8))))
     (pin "VSS" passive (at 77.8 419.5 0) (effects (font (size 0.8 0.8))))
+    (pin "VDDQ" input (at 77.8 421.0 0) (effects (font (size 0.8 0.8))))
   )
   (sheet (at 80.8 415.0) (size 12.0 15.0)
@@
     (pin "VDD" input (at 92.8 418.0 0) (effects (font (size 0.8 0.8))))
     (pin "VSS" passive (at 92.8 419.5 0) (effects (font (size 0.8 0.8))))
+    (pin "VDDQ" input (at 92.8 421.0 0) (effects (font (size 0.8 0.8))))
   )
   (sheet (at 95.8 415.0) (size 12.0 15.0)
@@
     (pin "VDD" input (at 107.8 418.0 0) (effects (font (size 0.8 0.8))))
     (pin "VSS" passive (at 107.8 419.5 0) (effects (font (size 0.8 0.8))))
+    (pin "VDDQ" input (at 107.8 421.0 0) (effects (font (size 0.8 0.8))))
   )
   (sheet (at 200.0 355.0) (size 12.0 15.0)
@@
     (pin "VDD" input (at 212.0 358.0 0) (effects (font (size 0.8 0.8))))
     (pin "VSS" passive (at 212.0 359.5 0) (effects (font (size 0.8 0.8))))
+    (pin "VDDQ" input (at 212.0 361.0 0) (effects (font (size 0.8 0.8))))
   )
   (sheet (at 215.0 355.0) (size 12.0 15.0)
@@
     (pin "VDD" input (at 227.0 358.0 0) (effects (font (size 0.8 0.8))))
     (pin "VSS" passive (at 227.0 359.5 0) (effects (font (size 0.8 0.8))))
+    (pin "VDDQ" input (at 227.0 361.0 0) (effects (font (size 0.8 0.8))))
   )
   (sheet (at 230.0 355.0) (size 12.0 15.0)
@@
     (pin "VDD" input (at 242.0 358.0 0) (effects (font (size 0.8 0.8))))
     (pin "VSS" passive (at 242.0 359.5 0) (effects (font (size 0.8 0.8))))
+    (pin "VDDQ" input (at 242.0 361.0 0) (effects (font (size 0.8 0.8))))
   )
   (sheet (at 245.0 355.0) (size 12.0 15.0)
@@
     (pin "VDD" input (at 257.0 358.0 0) (effects (font (size 0.8 0.8))))
     (pin "VSS" passive (at 257.0 359.5 0) (effects (font (size 0.8 0.8))))
+    (pin "VDDQ" input (at 257.0 361.0 0) (effects (font (size 0.8 0.8))))
   )
   (sheet (at 200.0 375.0) (size 12.0 15.0)
@@
     (pin "VDD" input (at 212.0 378.0 0) (effects (font (size 0.8 0.8))))
     (pin "VSS" passive (at 212.0 379.5 0) (effects (font (size 0.8 0.8))))
+    (pin "VDDQ" input (at 212.0 381.0 0) (effects (font (size 0.8 0.8))))
   )
   (sheet (at 215.0 375.0) (size 12.0 15.0)
@@
     (pin "VDD" input (at 227.0 378.0 0) (effects (font (size 0.8 0.8))))
     (pin "VSS" passive (at 227.0 379.5 0) (effects (font (size 0.8 0.8))))
+    (pin "VDDQ" input (at 227.0 381.0 0) (effects (font (size 0.8 0.8))))
   )
   (sheet (at 230.0 375.0) (size 12.0 15.0)
@@
     (pin "VDD" input (at 242.0 378.0 0) (effects (font (size 0.8 0.8))))
     (pin "VSS" passive (at 242.0 379.5 0) (effects (font (size 0.8 0.8))))
+    (pin "VDDQ" input (at 242.0 381.0 0) (effects (font (size 0.8 0.8))))
   )
   (sheet (at 245.0 375.0) (size 12.0 15.0)
@@
     (pin "VDD" input (at 257.0 378.0 0) (effects (font (size 0.8 0.8))))
     (pin "VSS" passive (at 257.0 379.5 0) (effects (font (size 0.8 0.8))))
+    (pin "VDDQ" input (at 257.0 381.0 0) (effects (font (size 0.8 0.8))))
   )
   (sheet (at 200.0 395.0) (size 12.0 15.0)
@@
     (pin "VDD" input (at 212.0 398.0 0) (effects (font (size 0.8 0.8))))
     (pin "VSS" passive (at 212.0 399.5 0) (effects (font (size 0.8 0.8))))
+    (pin "VDDQ" input (at 212.0 401.0 0) (effects (font (size 0.8 0.8))))
   )
   (sheet (at 215.0 395.0) (size 12.0 15.0)
@@
     (pin "VDD" input (at 227.0 398.0 0) (effects (font (size 0.8 0.8))))
     (pin "VSS" passive (at 227.0 399.5 0) (effects (font (size 0.8 0.8))))
+    (pin "VDDQ" input (at 227.0 401.0 0) (effects (font (size 0.8 0.8))))
   )
   (sheet (at 230.0 395.0) (size 12.0 15.0)
@@
     (pin "VDD" input (at 242.0 398.0 0) (effects (font (size 0.8 0.8))))
     (pin "VSS" passive (at 242.0 399.5 0) (effects (font (size 0.8 0.8))))
+    (pin "VDDQ" input (at 242.0 401.0 0) (effects (font (size 0.8 0.8))))
   )
   (sheet (at 245.0 395.0) (size 12.0 15.0)
@@
     (pin "VDD" input (at 257.0 398.0 0) (effects (font (size 0.8 0.8))))
     (pin "VSS" passive (at 257.0 399.5 0) (effects (font (size 0.8 0.8))))
+    (pin "VDDQ" input (at 257.0 401.0 0) (effects (font (size 0.8 0.8))))
   )
   (sheet (at 200.0 415.0) (size 12.0 15.0)
@@
     (pin "VDD" input (at 212.0 418.0 0) (effects (font (size 0.8 0.8))))
     (pin "VSS" passive (at 212.0 419.5 0) (effects (font (size 0.8 0.8))))
+    (pin "VDDQ" input (at 212.0 421.0 0) (effects (font (size 0.8 0.8))))
   )
   (sheet (at 215.0 415.0) (size 12.0 15.0)
@@
     (pin "VDD" input (at 227.0 418.0 0) (effects (font (size 0.8 0.8))))
     (pin "VSS" passive (at 227.0 419.5 0) (effects (font (size 0.8 0.8))))
+    (pin "VDDQ" input (at 227.0 421.0 0) (effects (font (size 0.8 0.8))))
   )
   (sheet (at 230.0 415.0) (size 12.0 15.0)
@@
     (pin "VDD" input (at 242.0 418.0 0) (effects (font (size 0.8 0.8))))
     (pin "VSS" passive (at 242.0 419.5 0) (effects (font (size 0.8 0.8))))
+    (pin "VDDQ" input (at 242.0 421.0 0) (effects (font (size 0.8 0.8))))
   )
   (sheet (at 245.0 415.0) (size 12.0 15.0)
@@
     (pin "VDD" input (at 257.0 418.0 0) (effects (font (size 0.8 0.8))))
     (pin "VSS" passive (at 257.0 419.5 0) (effects (font (size 0.8 0.8))))
+    (pin "VDDQ" input (at 257.0 421.0 0) (effects (font (size 0.8 0.8))))
   )
   (text "DUAL AI COMPUTE UNITS\nEach unit: AI SoC BGA (2500 pins) + 16x DDR5 DIMMs + 24-phase VRM\nTFLN Photonic Engine: 8ch RF differential per unit\nTotal: 1.6 Tbps aggregate optical bandwidth\nPCIe Gen6 x16 per unit (64 GT/s per lane)\nV_core: 0.8V, 1000A per unit (24-phase DrMOS)" (at 152.4 260.0 0) (effects (font (size 2.0 2.0)) (justify left)))
