File: LightRail_LPO_1.6T.kicad_sch (KiCad schematic)
At the start: 9 parts, among them J1 MPO-24, U1 TFLN_Mod_Gen3_8CH, U2 NeoPhotonics_1550nm_DFB, U3 Si5395A, U4 AD5684R, U5 MAX3669, U6 TPS7A2018, U7 TPS54360, U8 MPT5000

Commit message: fix(sch): add VDDQ hierarchical pin/label on AI_Core; README residual items
Devin Review flagged two doc/schematic gaps:

1. AI SoC VDDQ (DDR5 PHY I/O supply, 1.1 V) had a power_in pin on the
   AI_SoC symbol in AI_Core.kicad_sch but no hierarchical_label and no
   matching sheet pin on either AI_Core_Unit instance in the root
   schematic, so the rail was dangling at the hierarchy boundary. The
   VDDQ regulator (U31, TPS544C20) could not supply the SoC through the
   interface.

2. README residual items section still listed VDD_IO, TFLN_CLK_P/N, and
   VRM VID0/1/2 as missing -- these were added in Rev 4.1 and are
   already present, so the stale list would mislead the next engineer
   into adding duplicates and would hide the real missing pin (VDDQ).

Fixes: - Add hierarchical_label "VDDQ" (shape input) to AI_Core.kicad_sch
    alongside V_CORE and VDD_IO.
  - Add (pin "VDDQ" input ...) on both AI_Core_Unit0 and
    AI_Core_Unit1 sheet instances in LightRail_LPO_1.6T.kicad_sch,
    slotted between VDD_IO and TFLN_CLK_P with a 0.63 mm offset.
  - Rewrite README residual items to list only the genuinely missing
    DDR5 lane pins (DQ8..31, DQS1..3, DM1..3, CA4..13, CS1) and
    explicitly note that VDD_IO / VDDQ / TFLN_CLK / VID0..2 are done.
  - Add Rev 4.2 row to the revision history summarizing all the
    parse-fix / export / DRC / BOM fixes from this session.
Co-Authored-By: Bola Olatunji <bola.olatunji@ai.lightos.sh>
Other:
- sheet AI_Core_Unit0 ports: added VDDQ; removed none
- sheet AI_Core_Unit1 ports: added VDDQ; removed none
Changed lines of the file:
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@@
     (pin "PCIE_TX15N" bidirectional (at 110.8 294.68 0) (effects (font (size 1.0 1.0))))
     (pin "VDD_IO" input (at 50.8 300.40 180) (effects (font (size 1.0 1.0))))
+    (pin "VDDQ" input (at 50.8 301.03 180) (effects (font (size 1.0 1.0))))
     (pin "TFLN_CLK_P" output (at 50.8 301.67 180) (effects (font (size 1.0 1.0))))
     (pin "TFLN_CLK_N" output (at 50.8 302.94 180) (effects (font (size 1.0 1.0))))
@@
     (pin "PCIE_TX15N" bidirectional (at 260.0 294.68 0) (effects (font (size 1.0 1.0))))
     (pin "VDD_IO" input (at 200.0 300.40 180) (effects (font (size 1.0 1.0))))
+    (pin "VDDQ" input (at 200.0 301.03 180) (effects (font (size 1.0 1.0))))
     (pin "TFLN_CLK_P" output (at 200.0 301.67 180) (effects (font (size 1.0 1.0))))
     (pin "TFLN_CLK_N" output (at 200.0 302.94 180) (effects (font (size 1.0 1.0))))
