File: LightRail_LPO_1.6T.kicad_sch (KiCad schematic)
At the start: 9 parts, among them J1 MPO-24, U1 TFLN_Mod_Gen3_8CH, U2 NeoPhotonics_1550nm_DFB, U3 Si5395A, U4 AD5684R, U5 MAX3669, U6 TPS7A2018, U7 TPS54360, U8 MPT5000

Commit message: feat: HBM4 co-packaged memory migration (DDR5 -> HBM4 interposer)
Replace discrete DDR5-8800 DIMM fly-by subsystem with a co-packaged
NCE+HBM4-on-interposer topology per vendor reference (SK hynix /
Micron 12-Hi, 48 GB/stack, 8 Gbps/pin, 1024-bit bus).

PCB (LightRail_LPO_1.6T.kicad_pcb):
- Remove 8x DDR5 DIMM footprints (U202/U204/U206/U208 + U2102/..)
- Add 8x HBM4_Stack_11x11mm footprints (U103-U106 flanking U101,
  U203-U206 flanking U201) sitting on the co-packaged interposer
- Remove DDR5 CK fly-by segments on In2.Cu; nets 148-163 renamed
  DDR5_U{0,1}_* -> HBM4_U{0,1}_* (VDDC_S/VDDQL_S/VDDQ_S/VPP_S,
  REFCK_P/N, CATTRIP, PWR_GOOD, TCK/TMS/TDI/TDO)
- Silk text relabelled: 'DDR5-8800 Memory Bus (Fly-by Topology)'
  -> 'HBM4 Co-Packaged Memory (Advanced Interposer Path)'; central
  BGA value 'AI Compute Units (TFLN Photonics Enabled, NCE+HBM4
  Stack)'; bottom caption 'NCE+HBM4 Co-Packaged TFLN Photonics-
  integrated AI Compute Node (Based on MBoard [with 8x PCIe 5.0
  Slots])'
- Silicon interposer courtyard outlines added on F.Fab around each
  NCE+HBM4 module

Schematic:
- Memory.kicad_sch rewritten as HBM4_Stack_12Hi template (9 external
  side-channel pins + IEEE-1500 test bus)
- LightRail_LPO_1.6T.kicad_sch: 32 MEM_U*_D* DIMM sheets dropped;
  8 HBM4 stack sheets added; DDR5A_* sheet pins renamed HBM4_* on
  both AI_Core_Unit instances
- AI_Core.kicad_sch: DDR5A_* port names renamed HBM4_*
- .kicad_pro: net class DDR5_Data -> HBM4_Interposer

Fab:
- drc_custom.kicad_dru rewritten for HBM4 side-channel (REFCK 100 Ohm
  diff, IEEE-1500 50 Ohm SE, length 5-35 mm, P/N match +/-0.025 mm)
- generate_bom.py: 32 DDR5 DIMM entries -> 8 HBM4 stacks (SK hynix
  H56G48AT5DX117, marked 'TP' / DNP as vendor-supplied); VDDQ buck
  redescribed for HBM4; BOM.csv / BOM.md regenerated
- generate_pinouts.py: pinout_DDR5_DIMM.csv -> pinout_HBM4_Stack.csv;
  SoC BGA-2500 pinout table now lists VDDC/VDDQL/VDDQ/VPP HBM4 domains
  and flags the 1024x4 data bus as INTERPOSER-INTERN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
Other:
- removed sheet MEM_U0_D0
- removed sheet MEM_U0_D1
- removed sheet MEM_U0_D10
- removed sheet MEM_U0_D11
- removed sheet MEM_U0_D12
- removed sheet MEM_U0_D13
- removed sheet MEM_U0_D14
- removed sheet MEM_U0_D15
- removed sheet MEM_U0_D2
- removed sheet MEM_U0_D3
- removed sheet MEM_U0_D4
- removed sheet MEM_U0_D5
- removed sheet MEM_U0_D6
- removed sheet MEM_U0_D7
- removed sheet MEM_U0_D8
- removed sheet MEM_U0_D9
- removed sheet MEM_U1_D0
- removed sheet MEM_U1_D1
- removed sheet MEM_U1_D10
- removed sheet MEM_U1_D11
- removed sheet MEM_U1_D12
- removed sheet MEM_U1_D13
- removed sheet MEM_U1_D14
- removed sheet MEM_U1_D15
- removed sheet MEM_U1_D2
- removed sheet MEM_U1_D3
- removed sheet MEM_U1_D4
- removed sheet MEM_U1_D5
- removed sheet MEM_U1_D6
- removed sheet MEM_U1_D7
- removed sheet MEM_U1_D8
- removed sheet MEM_U1_D9
- added sheet HBM_U0_0 (Memory.kicad_sch)
- added sheet HBM_U0_1 (Memory.kicad_sch)
- added sheet HBM_U0_2 (Memory.kicad_sch)
- added sheet HBM_U0_3 (Memory.kicad_sch)
- added sheet HBM_U1_0 (Memory.kicad_sch)
- added sheet HBM_U1_1 (Memory.kicad_sch)
- added sheet HBM_U1_2 (Memory.kicad_sch)
- added sheet HBM_U1_3 (Memory.kicad_sch)
- sheet AI_Core_Unit0 ports: added HBM4_CATTRIP, HBM4_IEEE_TCK, HBM4_IEEE_TDI, HBM4_IEEE_TDO, HBM4_IEEE_TMS, HBM4_PWR_GOOD_0, HBM4_PWR_GOOD_1, HBM4_PWR_GOOD_2, HBM4_PWR_GOOD_3, HBM4_REFCK2_N, HBM4_REFCK2_P, HBM4_REFCK_N, HBM4_REFCK_P, HBM4_VDDC_S, HBM4_VDDQL_S, HBM4_VDDQ_S, HBM4_VPP_S; removed DDR5A_CA0, DDR5A_CA1, DDR5A_CA2, DDR5A_CA3, DDR5A_CK_N, DDR5A_CK_P, DDR5A_CS0, DDR5A_DQ0, DDR5A_DQ1, DDR5A_DQ2, DDR5A_DQ3, DDR5A_DQ4, DDR5A_DQ5, DDR5A_DQ6, DDR5A_DQ7, DDR5A_DQS0N, DDR5A_DQS0P
- sheet AI_Core_Unit1 ports: added HBM4_CATTRIP, HBM4_IEEE_TCK, HBM4_IEEE_TDI, HBM4_IEEE_TDO, HBM4_IEEE_TMS, HBM4_PWR_GOOD_0, HBM4_PWR_GOOD_1, HBM4_PWR_GOOD_2, HBM4_PWR_GOOD_3, HBM4_REFCK2_N, HBM4_REFCK2_P, HBM4_REFCK_N, HBM4_REFCK_P, HBM4_VDDC_S, HBM4_VDDQL_S, HBM4_VDDQ_S, HBM4_VPP_S; removed DDR5A_CA0, DDR5A_CA1, DDR5A_CA2, DDR5A_CA3, DDR5A_CK_N, DDR5A_CK_P, DDR5A_CS0, DDR5A_DQ0, DDR5A_DQ1, DDR5A_DQ2, DDR5A_DQ3, DDR5A_DQ4, DDR5A_DQ5, DDR5A_DQ6, DDR5A_DQ7, DDR5A_DQS0N, DDR5A_DQS0P
- note added: "DUAL AI COMPUTE UNITS Each unit: NCE BGA (2500 pins) + 4x HBM4 12-Hi stacks (co-packaged on silicon interposer) + 24-phase VRM TFLN Photonic Engine: 8ch RF differential per unit Total: 1.6 Tbps aggregate optical bandwidth PCIe Gen6 x16 per unit (64 GT/s per lane) V_core: 0.8V, 1000A per unit (24-phase DrMOS)"
- note removed: "DUAL AI COMPUTE UNITS Each unit: AI SoC BGA (2500 pins) + 16x DDR5 DIMMs + 24-phase VRM TFLN Photonic Engine: 8ch RF differential per unit Total: 1.6 Tbps aggregate optical bandwidth PCIe Gen6 x16 per unit (64 GT/s per lane) V_core: 0.8V, 1000A per unit (24-phase DrMOS)"
