File: Memory.kicad_sch (KiCad schematic)
At the start: 1 part, among them J201 DDR5_DIMM_288

Commit message: fix(pcb,sch,docs): Unit 1 In3 GND island; DDR5 diff Z 85->80 Ohm
Two Devin Review findings:

1. Unit 1 DDR5 CK (nets 160/161 on In2.Cu, x=90..149) had no lower
   reference plane. V_CORE_U0 on In3.Cu only covers x=5..78 (Unit 0
   region), and V_CORE_U1 is on In5/In6 — two dielectric layers below
   In2, too far to act as a return-path reference. Previously the
   deleted board-wide +12V zone on In3.Cu was accidentally serving
   that role; once it was removed for the V_CORE re-tasking, Unit 1
   signals on In2.Cu were left as one-sided microstrip referenced
   only to In1.Cu GND, which pushes their differential impedance to
   ~120 Ohm instead of the 80 Ohm target.

   Fix: added two GND fill zones (net 1) at In3.Cu and In4.Cu
   covering Unit 1 region (x=80..168, y=0..100). In3 GND restores
   the lower reference for DDR5 / PCIe signals on In2.Cu under
   Unit 1, giving a symmetric GND/GND stripline (vs Unit 0's
   asymmetric GND/V_CORE). In4 GND mirrors this for PDN plane
   continuity under Unit 1's BGA and keeps the stackup symmetric
   (V_CORE_U0 island on In3/In4 left half, GND island on In3/In4
   right half). Updated docs/Stackup.md §2 Asymmetric stripline
   note to document the two-region reference strategy explicitly.

2. Memory.kicad_sch said '85 Ohm differential for DQ/DQS' (lines
   13 and 159) while docs/Stackup.md:79 specifies 80 Ohm diff for
   DDR5_Data. The 5 Ohm gap matters because a 2D field solver will
   produce different trace widths/gaps for 80 vs 85 Ohm — a fab
   following one doc will fail the other's spec. Standardised on
   80 Ohm diff / 40 Ohm SE (JEDEC JESD79-5 baseline for DDR5-5600)
   in both Memory.kicad_sch comment lines.

Co-Authored-By: Bola Olatunji <bola.olatunji@ai.lightos.sh>
Other:
- note added: "DDR5 MEMORY INTERFACE DDR5-5600 DIMM Slot (288-pin) Fly-by Topology: CK slightly longer than C/A (JEDEC) Impedance: 80 Ohm differential for DQ/DQS (40 Ohm SE) Duplicate this sheet for each DIMM slot"
- note removed: "DDR5 MEMORY INTERFACE DDR5-5600 DIMM Slot (288-pin) Fly-by Topology: CK slightly longer than C/A (JEDEC) Impedance: 85 Ohm differential for DQ/DQS Duplicate this sheet for each DIMM slot"
Changed lines of the file:
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@@
     (comment 2 "JEDEC DDR5 compliant C/A bus routing")
     (comment 3 "Duplicate this sheet for each DIMM (up to 16 per compute unit)")
-    (comment 4 "85 Ohm differential impedance for DQ/DQS")
+    (comment 4 "80 Ohm differential impedance for DQ/DQS (40 Ohm SE), matches docs/Stackup.md")
   )
   (symbol (lib_id "LightRail:DDR5_DIMM_288") (at 152.4 127.0 0) (unit 1) (in_bom yes) (on_board yes)
@@
   (hierarchical_label "VDDQ" (shape input) (at 40.64 43.0 180) (effects (font (size 1.27 1.27))))
   (hierarchical_label "VSS" (shape passive) (at 40.64 46.0 180) (effects (font (size 1.27 1.27))))
-  (text "DDR5 MEMORY INTERFACE\nDDR5-5600 DIMM Slot (288-pin)\nFly-by Topology: CK slightly longer than C/A (JEDEC)\nImpedance: 85 Ohm differential for DQ/DQS\nDuplicate this sheet for each DIMM slot" (at 152.4 30.48 0) (effects (font (size 2.0 2.0)) (justify left)))
+  (text "DDR5 MEMORY INTERFACE\nDDR5-5600 DIMM Slot (288-pin)\nFly-by Topology: CK slightly longer than C/A (JEDEC)\nImpedance: 80 Ohm differential for DQ/DQS (40 Ohm SE)\nDuplicate this sheet for each DIMM slot" (at 152.4 30.48 0) (effects (font (size 2.0 2.0)) (justify left)))
 ) ;; end kicad_sch
