File: Memory.kicad_sch (KiCad schematic)
At the start: 1 part, among them J201 DDR5_DIMM_288

Commit message: feat: HBM4 co-packaged memory migration (DDR5 -> HBM4 interposer)
Replace discrete DDR5-8800 DIMM fly-by subsystem with a co-packaged
NCE+HBM4-on-interposer topology per vendor reference (SK hynix /
Micron 12-Hi, 48 GB/stack, 8 Gbps/pin, 1024-bit bus).

PCB (LightRail_LPO_1.6T.kicad_pcb):
- Remove 8x DDR5 DIMM footprints (U202/U204/U206/U208 + U2102/..)
- Add 8x HBM4_Stack_11x11mm footprints (U103-U106 flanking U101,
  U203-U206 flanking U201) sitting on the co-packaged interposer
- Remove DDR5 CK fly-by segments on In2.Cu; nets 148-163 renamed
  DDR5_U{0,1}_* -> HBM4_U{0,1}_* (VDDC_S/VDDQL_S/VDDQ_S/VPP_S,
  REFCK_P/N, CATTRIP, PWR_GOOD, TCK/TMS/TDI/TDO)
- Silk text relabelled: 'DDR5-8800 Memory Bus (Fly-by Topology)'
  -> 'HBM4 Co-Packaged Memory (Advanced Interposer Path)'; central
  BGA value 'AI Compute Units (TFLN Photonics Enabled, NCE+HBM4
  Stack)'; bottom caption 'NCE+HBM4 Co-Packaged TFLN Photonics-
  integrated AI Compute Node (Based on MBoard [with 8x PCIe 5.0
  Slots])'
- Silicon interposer courtyard outlines added on F.Fab around each
  NCE+HBM4 module

Schematic:
- Memory.kicad_sch rewritten as HBM4_Stack_12Hi template (9 external
  side-channel pins + IEEE-1500 test bus)
- LightRail_LPO_1.6T.kicad_sch: 32 MEM_U*_D* DIMM sheets dropped;
  8 HBM4 stack sheets added; DDR5A_* sheet pins renamed HBM4_* on
  both AI_Core_Unit instances
- AI_Core.kicad_sch: DDR5A_* port names renamed HBM4_*
- .kicad_pro: net class DDR5_Data -> HBM4_Interposer

Fab:
- drc_custom.kicad_dru rewritten for HBM4 side-channel (REFCK 100 Ohm
  diff, IEEE-1500 50 Ohm SE, length 5-35 mm, P/N match +/-0.025 mm)
- generate_bom.py: 32 DDR5 DIMM entries -> 8 HBM4 stacks (SK hynix
  H56G48AT5DX117, marked 'TP' / DNP as vendor-supplied); VDDQ buck
  redescribed for HBM4; BOM.csv / BOM.md regenerated
- generate_pinouts.py: pinout_DDR5_DIMM.csv -> pinout_HBM4_Stack.csv;
  SoC BGA-2500 pinout table now lists VDDC/VDDQL/VDDQ/VPP HBM4 domains
  and flags the 1024x4 data bus as INTERPOSER-INTERN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
Parts:
- U?: renamed from J201; value DDR5_DIMM_288 -> HBM4_12Hi_48GB; footprint LightRail:DDR5_DIMM_288pin -> LightRail:HBM4_Stack_11x11mm; symbol LightRail:DDR5_DIMM_288 -> LightRail:HBM4_Stack_12Hi
Other:
- note added: "HBM4 CO-PACKAGED MEMORY STACK 12-Hi 48 GB (HBM4) Data bus (1024 lanes @ 8 Gbps/pin) is INTERNAL to the silicon interposer. PCB sees only power, REFCK, CATTRIP, PWR_GOOD, IEEE 1500 test bus. Instantiate once per stack (4 per compute unit, 8 total per board)."
- note removed: "DDR5 MEMORY INTERFACE DDR5-5600 DIMM Slot (288-pin) Fly-by Topology: CK slightly longer than C/A (JEDEC) Impedance: 80 Ohm differential for DQ/DQS (40 Ohm SE) Duplicate this sheet for each DIMM slot"
- title: DDR5 Memory Interface -> HBM4 Co-Packaged Memory Stack
